File: Proj_5/8086_Demuxing.sch (KiCad schematic (older format))
At the start: 7 parts

Commit message: Buffered and Demultiplexed Address/Data Bus
Connections:
- net labels added: A0, A1, A10, A11, A12, A13, A14, A15, A16, A17, A18, A19, A2, A3, A4, A5, A6, A7, A8, A9, D0, D1, D10, D11, D12, D13, D14, D15, D2, D3, D4, D5, D6, D7, D8, D9, GND, M~IO, VCC, ~BHE, ~RD, ~WR
- wire segments 29 -> 221
- no-connect marks 0 -> 6
Other:
- note added: "Needs Power/Clarifications on Data bus buffer select pins 4/21\n"
- moved on the sheet: U?

Commit message: Please work
Parts:
- U?: symbol MCU_Intel:8086_Min_Mode -> Proj_5-rescue:8086_Min_Mode-MCU_Intel
Changed lines of the file:
@@
 $EndDescr
 $Comp
-L MCU_Intel:8086_Min_Mode U?
+L Proj_5-rescue:8086_Min_Mode-MCU_Intel U?
 U 1 1 5E9F413F
 P 7850 8700
+AR Path="/5E9F413F" Ref="U?"  Part="1"
+AR Path="/5E9F3A3D/5E9F413F" Ref="U?"  Part="1"
 F 0 "U?" H 7850 10681 50  0000 C CNN
 F 1 "8086_Min_Mode" H 7850 10590 50  0000 C CNN
