File: Proj_5/8086_Demuxing.sch (KiCad schematic (older format))
At the start: 8 parts, among them U19 8086_Min_Mode, U20 74LS373, U21 74LS373, U22 74LS244, U23 74LS373, U24 74LS245, U25 74LS245

Commit message: Rerouted Ext Wires, UART Mostly Complete, All Headers Added
Parts:
- added J?: Conn_02x30_Top_Bottom, symbol Connector_Generic:Conn_02x30_Top_Bottom
Connections:
- net A0: now also J?.31 (Pin_31)
- net A1: now also J?.32 (Pin_32)
- net A10: now also J?.41 (Pin_41)
- net A11: now also J?.42 (Pin_42)
- net A12: now also J?.43 (Pin_43)
- net A13: now also J?.44 (Pin_44)
- net A14: now also J?.45 (Pin_45)
- net A15: now also J?.46 (Pin_46)
- net A16: now also J?.47 (Pin_47)
- net A17: now also J?.48 (Pin_48)
- net A18: now also J?.49 (Pin_49)
- net A19: now also J?.50 (Pin_50)
- net A2: now also J?.33 (Pin_33)
- net A3: now also J?.34 (Pin_34)
- net A4: now also J?.35 (Pin_35)
- net A5: now also J?.36 (Pin_36)
- net A6: now also J?.37 (Pin_37)
- net A7: now also J?.38 (Pin_38)
- net A8: now also J?.39 (Pin_39)
- net A9: now also J?.40 (Pin_40)
- net D0: now also J?.15 (Pin_15)
- net D1: now also J?.16 (Pin_16)
- net D10: now also J?.25 (Pin_25)
- net D11: now also J?.26 (Pin_26)
- net D12: now also J?.27 (Pin_27)
- net D13: now also J?.28 (Pin_28)
- net D14: now also J?.29 (Pin_29)
- net D15: now also J?.30 (Pin_30)
- net D2: now also J?.17 (Pin_17)
- net D3: now also J?.18 (Pin_18)
- net D4: now also J?.19 (Pin_19)
- net D5: now also J?.20 (Pin_20)
- net D6: now also J?.21 (Pin_21)
- net D7: now also J?.22 (Pin_22)
- net D8: now also J?.23 (Pin_23)
- net D9: now also J?.24 (Pin_24)
- net GND: now also J?.1 (Pin_1), J?.10 (Pin_10), J?.11 (Pin_11), J?.12 (Pin_12), J?.13 (Pin_13), J?.14 (Pin_14), J?.2 (Pin_2), J?.3 (Pin_3), J?.4 (Pin_4), J?.5 (Pin_5), J?.6 (Pin_6), J?.60 (Pin_60), J?.7 (Pin_7), J?.8 (Pin_8), J?.9 (Pin_9)
- net M~IO: now also J?.54 (Pin_54)
- net ~BHE: now also J?.51 (Pin_51)
- net ~RD: now also J?.52 (Pin_52)
- net ~WR: now also J?.53 (Pin_53)
- net NMI_IN: now reaches U19.17 (NMI)
- net at U19.18 (INTR): now also J?.58 (Pin_58)
- net at U19.22 (READY): now also J?.59 (Pin_59)
- net at U19.23 (~TEST~): now also J?.57 (Pin_57)
- net at U19.30 (HLDA): now also J?.56 (Pin_56)
- net at U19.31 (HOLD): now also J?.55 (Pin_55)

Commit message: Remaining LED Components Added, Final pins added to headers.
Connections:
- net GND: no longer J?.60 (Pin_60)
- net VCC: now also C14.2, U19.40 (VCC), U20.20 (VCC), U21.20 (VCC), U23.20 (VCC), U24.20 (VCC), U25.20 (VCC)
- net at U19.24 (~INTA~): now also U22.8 (I3a)
- net at U22.12 (O3a): now also J?.60 (Pin_60)
Other:
- note removed: "Needs Power/Clarifications on Data bus buffer select pins 4/21\n"
Changed lines of the file:
@@
 	0    -1   -1   0
 $EndComp
-Text Notes 15850 7100 0    79   ~ 0
-Needs Power/Clarifications on Data bus buffer select pins 4/21\n
 Wire Wire Line
 	8550 9950 10400 9950
@@
 	7850 6550 7850 6900
 Wire Wire Line
-	7850 6100 7850 6550
+	7850 6100 7850 6150
 Connection ~ 7850 6550
 $Comp
@@
 	11650 3750 11650 3350
 Wire Wire Line
-	11550 3350 11100 3350
-Wire Wire Line
-	11100 3350 11100 3300
-$Comp
-L power:GND #PWR?
-U 1 1 5F0E7C3D
-P 11100 3300
-F 0 "#PWR?" H 11100 3050 50  0001 C CNN
-F 1 "GND" H 11105 3127 50  0000 C CNN
-F 2 "" H 11100 3300 50  0001 C CNN
-F 3 "" H 11100 3300 50  0001 C CNN
-	1    11100 3300
-	-1   0    0    1
-$EndComp
-Wire Wire Line
 	20450 8900 20450 500
 Wire Wire Line
@@
 $EndComp
 Connection ~ 14450 2500
+$Comp
+L power:VCC #PWR?
+U 1 1 5EF73B7F
+P 7850 6100
+F 0 "#PWR?" H 7850 5950 50  0001 C CNN
+F 1 "VCC" H 7867 6273 50  0000 C CNN
+F 2 "" H 7850 6100 50  0001 C CNN
+F 3 "" H 7850 6100 50  0001 C CNN
+	1    7850 6100
+	1    0    0    -1
+$EndComp
+Wire Wire Line
+	9500 7150 9500 7600
+$Comp
+L power:VCC #PWR?
+U 1 1 5EF74C0E
+P 9500 7150
+F 0 "#PWR?" H 9500 7000 50  0001 C CNN
+F 1 "VCC" H 9517 7323 50  0000 C CNN
+F 2 "" H 9500 7150 50  0001 C CNN
+F 3 "" H 9500 7150 50  0001 C CNN
+	1    9500 7150
+	1    0    0    -1
+$EndComp
+Wire Wire Line
+	12100 7150 12100 7600
+$Comp
+L power:VCC #PWR?
+U 1 1 5EF9EA73
+P 12100 7150
+F 0 "#PWR?" H 12100 7000 50  0001 C CNN
+F 1 "VCC" H 12117 7323 50  0000 C CNN
+F 2 "" H 12100 7150 50  0001 C CNN
+F 3 "" H 12100 7150 50  0001 C CNN
+	1    12100 7150
+	1    0    0    -1
+$EndComp
+Wire Wire Line
+	16900 7600 17350 7600
+$Comp
+L power:VCC #PWR?
+U 1 1 5EFC96F5
+P 16900 7600
+F 0 "#PWR?" H 16900 7450 50  0001 C CNN
+F 1 "VCC" H 16917 7773 50  0000 C CNN
+F 2 "" H 16900 7600 50  0001 C CNN
+F 3 "" H 16900 7600 50  0001 C CNN
+	1    16900 7600
+	0    -1   -1   0
+$EndComp
+Wire Wire Line
+	16400 9400 15950 9400
+$Comp
+L power:VCC #PWR?
+U 1 1 5EFF3F9C
+P 16400 9400
+F 0 "#PWR?" H 16400 9250 50  0001 C CNN
+F 1 "VCC" H 16417 9573 50  0000 C CNN
+F 2 "" H 16400 9400 50  0001 C CNN
+F 3 "" H 16400 9400 50  0001 C CNN
+	1    16400 9400
+	0    1    1    0
+$EndComp
+Wire Wire Line
+	10850 10650 11300 10650
+$Comp
+L power:VCC #PWR?
+U 1 1 5F01F222
+P 10850 10650
+F 0 "#PWR?" H 10850 10500 50  0001 C CNN
+F 1 "VCC" H 10867 10823 50  0000 C CNN
+F 2 "" H 10850 10650 50  0001 C CNN
+F 3 "" H 10850 10650 50  0001 C CNN
+	1    10850 10650
+	0    -1   -1   0
+$EndComp
+Wire Wire Line
+	9750 3950 10200 3950
+$Comp
+L power:VCC #PWR?
+U 1 1 5F04A79B
+P 9750 3950
+F 0 "#PWR?" H 9750 3800 50  0001 C CNN
+F 1 "VCC" H 9767 4123 50  0000 C CNN
+F 2 "" H 9750 3950 50  0001 C CNN
+F 3 "" H 9750 3950 50  0001 C CNN
+	1    9750 3950
+	0    -1   -1   0
+$EndComp
+$Comp
+L power:PWR_FLAG #FLG?
+U 1 1 5F179D43
+P 7850 6150
+AR Path="/5EA045EA/5F179D43" Ref="#FLG?"  Part="1"
+AR Path="/5EA98353/5EA34234/5F179D43" Ref="#FLG?"  Part="1"
+AR Path="/5E9F3A3D/5F179D43" Ref="#FLG?"  Part="1"
+F 0 "#FLG?" H 7850 6225 50  0001 C CNN
+F 1 "PWR_FLAG" V 7850 6277 50  0000 L CNN
+F 2 "" H 7850 6150 50  0001 C CNN
+F 3 "~" H 7850 6150 50  0001 C CNN
+	1    7850 6150
+	0    1    1    0
+$EndComp
+Connection ~ 7850 6150
+Wire Wire Line
+	7850 6150 7850 6550
+Wire Wire Line
+	8550 10250 10100 10250
+Wire Wire Line
+	10100 10250 10100 11250
+Wire Wire Line
+	10100 11250 10750 11250
+Wire Wire Line
+	11750 11250 12450 11250
+Wire Wire Line
+	12450 11250 12450 13150
+Wire Wire Line
+	12450 13150 4200 13150
+Wire Wire Line
+	4200 13150 4200 3800
+Wire Wire Line
+	4200 3800 11550 3800
+Wire Wire Line
+	11550 3800 11550 3350
 $EndSCHEMATC

Commit message: Added Power Flags, finished no connects.
Parts:
- gave numbers to parts that had none: 1
Connections:
- net at U19.18 (INTR): now also J6.55 (Pin_55); no longer J6.58 (Pin_58)
- net at U19.22 (READY): now also J6.56 (Pin_56); no longer J6.59 (Pin_59)
- net at U19.23 (~TEST~): no longer J6.57 (Pin_57)
- net at U19.30 (HLDA): no longer J6.56 (Pin_56)
- net at U19.31 (HOLD): no longer J6.55 (Pin_55)
- net at U22.12 (O3a): now also J6.57 (Pin_57); no longer J6.60 (Pin_60)
- no-connect marks 6 -> 21

Commit message: Finished Most of power flags, power connector header, added hierachical pins to a few sheets.
Parts:
- added C?: 100uF, symbol Device:C
- added J?: Conn_01x02, symbol Connector_Generic:Conn_01x02
Connections:
- net GND: now also C?.1, J?.1 (Pin_1)
- net VCC: now also C?.2, J?.2 (Pin_2)
Changed lines of the file:
@@
 $Descr A2 23386 16535
 encoding utf-8
-Sheet 8 10
+Sheet 7 10
 Title ""
 Date ""
@@
 NoConn ~ 11650 3350
 NoConn ~ 11550 3350
+$Comp
+L Connector_Generic:Conn_01x02 J?
+U 1 1 5EEC8283
+P 3250 1500
+F 0 "J?" H 3168 1175 50  0000 C CNN
+F 1 "Conn_01x02" H 3168 1266 50  0000 C CNN
+F 2 "" H 3250 1500 50  0001 C CNN
+F 3 "~" H 3250 1500 50  0001 C CNN
+	1    3250 1500
+	-1   0    0    1
+$EndComp
+Wire Wire Line
+	4000 1200 4000 1250
+$Comp
+L power:VCC #PWR?
+U 1 1 5EEC8F27
+P 4000 1200
+F 0 "#PWR?" H 4000 1050 50  0001 C CNN
+F 1 "VCC" H 4017 1373 50  0000 C CNN
+F 2 "" H 4000 1200 50  0001 C CNN
+F 3 "" H 4000 1200 50  0001 C CNN
+	1    4000 1200
+	1    0    0    -1
+$EndComp
+$Comp
+L power:PWR_FLAG #FLG?
+U 1 1 5EEC8F2D
+P 4000 1250
+AR Path="/5EA045EA/5EEC8F2D" Ref="#FLG?"  Part="1"
+AR Path="/5EA98353/5EA34234/5EEC8F2D" Ref="#FLG?"  Part="1"
+AR Path="/5E9F3A3D/5EEC8F2D" Ref="#FLG?"  Part="1"
+F 0 "#FLG?" H 4000 1325 50  0001 C CNN
+F 1 "PWR_FLAG" V 4000 1377 50  0000 L CNN
+F 2 "" H 4000 1250 50  0001 C CNN
+F 3 "~" H 4000 1250 50  0001 C CNN
+	1    4000 1250
+	0    1    1    0
+$EndComp
+Wire Wire Line
+	4000 1250 4000 1400
+Connection ~ 4000 1250
+$Comp
+L Device:C C?
+U 1 1 5EFA8610
+P 4500 1500
+AR Path="/5EA98353/5EFA8610" Ref="C?"  Part="1"
+AR Path="/5E9F3A3D/5EFA8610" Ref="C?"  Part="1"
+F 0 "C?" V 4248 1500 50  0000 C CNN
+F 1 "100uF" V 4339 1500 50  0000 C CNN
+F 2 "" H 4538 1350 50  0001 C CNN
+F 3 "~" H 4500 1500 50  0001 C CNN
+	1    4500 1500
+	-1   0    0    1
+$EndComp
+$Comp
+L power:GND #PWR?
+U 1 1 5EFA8616
+P 4500 1700
+F 0 "#PWR?" H 4500 1450 50  0001 C CNN
+F 1 "GND" H 4505 1527 50  0000 C CNN
+F 2 "" H 4500 1700 50  0001 C CNN
+F 3 "" H 4500 1700 50  0001 C CNN
+	1    4500 1700
+	1    0    0    -1
+$EndComp
+$Comp
+L power:PWR_FLAG #FLG?
+U 1 1 5EFA861C
+P 4500 1700
+AR Path="/5EAF7226/5EFA861C" Ref="#FLG?"  Part="1"
+AR Path="/5E9F3A3D/5EFA861C" Ref="#FLG?"  Part="1"
+F 0 "#FLG?" H 4500 1775 50  0001 C CNN
+F 1 "PWR_FLAG" V 4500 1828 50  0000 L CNN
+F 2 "" H 4500 1700 50  0001 C CNN
+F 3 "~" H 4500 1700 50  0001 C CNN
+	1    4500 1700
+	0    -1   -1   0
+$EndComp
+Wire Wire Line
+	4500 1350 4300 1350
+Wire Wire Line
+	4300 1350 4300 1400
+Wire Wire Line
+	3450 1400 4000 1400
+Connection ~ 4000 1400
+Wire Wire Line
+	4000 1400 4300 1400
+Wire Wire Line
+	4150 1500 4150 1650
+Wire Wire Line
+	4150 1650 4500 1650
+Wire Wire Line
+	3450 1500 4150 1500
+Wire Wire Line
+	4500 1650 4500 1700
+Connection ~ 4500 1650
+Connection ~ 4500 1700
 $EndSCHEMATC

Commit message: Power Flags
Parts:
- gave numbers to parts that had none: 2

Commit message: 11 errors left
Connections:
- net GND: now also U20.1 (OE)
- net VCC: now also U22.20 (VCC)
Changed lines of the file:
@@
 L power:GND #PWR09
 U 1 1 5EA86357
-P 8350 6550
-F 0 "#PWR09" H 8350 6300 50  0001 C CNN
-F 1 "GND" H 8355 6377 50  0000 C CNN
-F 2 "" H 8350 6550 50  0001 C CNN
-F 3 "" H 8350 6550 50  0001 C CNN
-	1    8350 6550
+P 8550 6550
+F 0 "#PWR09" H 8550 6300 50  0001 C CNN
+F 1 "GND" H 8555 6377 50  0000 C CNN
+F 2 "" H 8550 6550 50  0001 C CNN
+F 3 "" H 8550 6550 50  0001 C CNN
+	1    8550 6550
 	0    -1   -1   0
 $EndComp
@@
 	-1   0    0    1
 $EndComp
-Wire Wire Line
-	10850 10650 11300 10650
 $Comp
 L power:VCC #PWR087
@@
 Wire Wire Line
 	4000 1200 4000 1400
+Wire Wire Line
+	8550 6550 8350 6550
+Wire Wire Line
+	10850 10650 11250 10650
+Wire Wire Line
+	9700 5250 9700 5500
+$Comp
+L power:GND #PWR0132
+U 1 1 5EFCFA5B
+P 9700 5500
+F 0 "#PWR0132" H 9700 5250 50  0001 C CNN
+F 1 "GND" H 9705 5327 50  0000 C CNN
+F 2 "" H 9700 5500 50  0001 C CNN
+F 3 "" H 9700 5500 50  0001 C CNN
+	1    9700 5500
+	1    0    0    -1
+$EndComp
 $EndSCHEMATC

Commit message: 1 Error Remains
Connections:
- net INTR_IN: now reaches J6.55 (Pin_55), U19.18 (INTR)
- net ~INTA_OUT: now reaches J6.57 (Pin_57), U22.12 (O3a)
Changed lines of the file:
@@
 	3500 3500 3500 13250
 Wire Wire Line
-	7150 8100 3900 8100
+	7150 8100 6650 8100
 Wire Wire Line
 	3900 8100 3900 3700
@@
 	1    0    0    -1
 $EndComp
+$Comp
+L power:VCC #PWR0133
+U 1 1 5EBBDB8A
+P 5050 950
+F 0 "#PWR0133" H 5050 800 50  0001 C CNN
+F 1 "VCC" H 5067 1123 50  0000 C CNN
+F 2 "" H 5050 950 50  0001 C CNN
+F 3 "" H 5050 950 50  0001 C CNN
+	1    5050 950
+	1    0    0    -1
+$EndComp
+$Comp
+L power:GND #PWR0134
+U 1 1 5EBEBF8D
+P 5500 1150
+F 0 "#PWR0134" H 5500 900 50  0001 C CNN
+F 1 "GND" H 5505 977 50  0000 C CNN
+F 2 "" H 5500 1150 50  0001 C CNN
+F 3 "" H 5500 1150 50  0001 C CNN
+	1    5500 1150
+	1    0    0    -1
+$EndComp
+$Comp
+L power:PWR_FLAG #FLG0101
+U 1 1 5EC1A8E6
+P 5050 1150
+F 0 "#FLG0101" H 5050 1225 50  0001 C CNN
+F 1 "PWR_FLAG" H 5050 1323 50  0000 C CNN
+F 2 "" H 5050 1150 50  0001 C CNN
+F 3 "~" H 5050 1150 50  0001 C CNN
+	1    5050 1150
+	-1   0    0    1
+$EndComp
+$Comp
+L power:PWR_FLAG #FLG0102
+U 1 1 5EC1BC9D
+P 5500 950
+F 0 "#FLG0102" H 5500 1025 50  0001 C CNN
+F 1 "PWR_FLAG" H 5500 1123 50  0000 C CNN
+F 2 "" H 5500 950 50  0001 C CNN
+F 3 "~" H 5500 950 50  0001 C CNN
+	1    5500 950
+	1    0    0    -1
+$EndComp
+Wire Wire Line
+	5500 950  5500 1150
+Wire Wire Line
+	5050 950  5050 1150
+Text HLabel 12900 11250 2    50   Output ~ 0
+~INTA_OUT
+Text HLabel 6450 8000 0    50   Input ~ 0
+INTR_IN
+Wire Wire Line
+	12450 11250 12900 11250
+Connection ~ 12450 11250
+Wire Wire Line
+	6450 8000 6650 8000
+Wire Wire Line
+	6650 8000 6650 8100
+Connection ~ 6650 8100
+Wire Wire Line
+	6650 8100 3900 8100
 $EndSCHEMATC
