File: Proj_5/CMOS-28F010s.sch (KiCad schematic (older format))
At the start: 8 parts

Commit message: Please work
Parts:
- removed U? (x7): 28F010, 28F010, symbol 28F010:28F010
- added U11, U4, U5, U6, U7, U8, U9: 28F010, 28F010, symbol 28F010:28F010
- gave numbers to parts that had none: 1
Connections:
- net GND: now reaches U10.16 (VSS)
- net GND: now also U11.16 (VSS), U4.16 (VSS), U5.16 (VSS), U6.16 (VSS), U7.16 (VSS), U8.16 (VSS), U9.16 (VSS)
- net +5V: now reaches U10.32 (VCC)
- net +5V: now also U11.32 (VCC), U4.32 (VCC), U5.32 (VCC), U6.32 (VCC), U7.32 (VCC), U8.32 (VCC), U9.32 (VCC)
- no-connect marks 0 -> 10
Other:
- moved on the sheet: U10
