File: Proj_5/CMOS-28F010s.sch (KiCad schematic (older format))
At the start: 4 parts, among them U4 28F010

Commit message: Changed Addressing Again
Parts:
- added U?: PAL16L8, symbol Logic_Programmable:PAL16L8
Connections:
- net A10: now also U4.23 (A10), U?.23 (A10); no longer U4.5 (A7), U?.5 (A7)
- net A11: now also U4.25 (A11), U?.25 (A11); no longer U4.27 (A8), U?.27 (A8)
- net A12: now also U4.4 (A12), U?.4 (A12); no longer U4.26 (A9), U?.26 (A9)
- net A13: now also U4.28 (A13), U?.28 (A13); no longer U4.23 (A10), U?.23 (A10)
- net A14: now also U4.29 (A14), U?.29 (A14); no longer U4.25 (A11), U?.25 (A11)
- net A15: now also U4.3 (A15), U?.3 (A15); no longer U4.4 (A12), U?.4 (A12)
- net A16: now also U4.2 (A16), U?.2 (A16); no longer U4.28 (A13), U?.28 (A13)
- net A17: now also U?.17 (I03); no longer U4.29 (A14), U?.29 (A14)
- net A18: now also U?.18 (IO2); no longer U4.3 (A15), U?.3 (A15)
- net A19: now also U?.19 (IO1); no longer U4.2 (A16), U?.2 (A16)
- net A3: now also U4.9 (A3), U?.9 (A3); no longer U4.12 (A0), U?.12 (A0)
- net A4: now also U4.8 (A4), U?.8 (A4); no longer U4.11 (A1), U?.11 (A1)
- net A5: now also U4.7 (A5), U?.7 (A5); no longer U4.10 (A2), U?.10 (A2)
- net A6: now also U4.6 (A6), U?.6 (A6); no longer U4.9 (A3), U?.9 (A3)
- net A7: now also U4.5 (A7), U?.5 (A7); no longer U4.8 (A4), U?.8 (A4)
- net A8: now also U4.27 (A8), U?.27 (A8); no longer U4.7 (A5), U?.7 (A5)
- net A9: now also U4.26 (A9), U?.26 (A9); no longer U4.6 (A6), U?.6 (A6)
- net ~BHE: now also U4.12 (A0), U?.12 (A0), U?.15 (IO5); no longer U4.22 (CE)
- net ~BLE: now also U?.16 (IO4); no longer U?.22 (CE)
- new net: U?.2 (I2), U?.22 (CE)
- new net: U4.22 (CE), U?.1 (I1)
- new net A1: U4.11 (A1), U?.11 (A1)
- new net A2: U4.10 (A2), U?.10 (A2)
Other:
- note added: "Address Range: DFFFFh - FFFFFh (917503 - 1048575 dec)"
Changed lines of the file:
@@
 Wire Wire Line
 	7350 3300 6850 3300
-Text HLabel 3600 3700 0    50   Input ~ 0
-A3
-Text HLabel 3600 3600 0    50   Input ~ 0
-A4
-Text HLabel 3600 3500 0    50   Input ~ 0
-A5
-Text HLabel 3600 3400 0    50   Input ~ 0
-A6
-Text HLabel 3600 3300 0    50   Input ~ 0
-A7
-Text HLabel 3600 3200 0    50   Input ~ 0
-A8
-Text HLabel 3600 3100 0    50   Input ~ 0
-A9
-Text HLabel 3600 3000 0    50   Input ~ 0
-A10
-Text HLabel 3600 2900 0    50   Input ~ 0
-A15
-Text HLabel 3600 2800 0    50   Input ~ 0
-A18
-Text HLabel 3600 2700 0    50   Input ~ 0
-A19
-Text HLabel 7350 2900 2    50   Input ~ 0
-A17
-Text HLabel 7350 3000 2    50   Input ~ 0
-A16
-Text HLabel 7350 3100 2    50   Input ~ 0
-A11
-Text HLabel 7350 3200 2    50   Input ~ 0
-A12
-Text HLabel 7350 3300 2    50   Input ~ 0
-A14
-Text HLabel 7350 3500 2    50   Input ~ 0
-A13
 Text HLabel 7250 3700 2    50   BiDi ~ 0
 D15
@@
 Wire Wire Line
 	7350 6000 6850 6000
-Text HLabel 3600 6400 0    50   Input ~ 0
-A3
-Text HLabel 3600 6300 0    50   Input ~ 0
-A4
-Text HLabel 3600 6200 0    50   Input ~ 0
-A5
-Text HLabel 3600 6100 0    50   Input ~ 0
-A6
-Text HLabel 3600 6000 0    50   Input ~ 0
-A7
-Text HLabel 3600 5900 0    50   Input ~ 0
-A8
-Text HLabel 3600 5800 0    50   Input ~ 0
-A9
-Text HLabel 3600 5700 0    50   Input ~ 0
-A10
-Text HLabel 3600 5600 0    50   Input ~ 0
-A15
-Text HLabel 3600 5500 0    50   Input ~ 0
-A18
-Text HLabel 3600 5400 0    50   Input ~ 0
-A19
-Text HLabel 7350 5600 2    50   Input ~ 0
-A17
-Text HLabel 7350 5700 2    50   Input ~ 0
-A16
-Text HLabel 7350 5800 2    50   Input ~ 0
-A11
-Text HLabel 7350 5900 2    50   Input ~ 0
-A12
-Text HLabel 7350 6000 2    50   Input ~ 0
-A14
-Text HLabel 7350 6200 2    50   Input ~ 0
-A13
 Text HLabel 7250 6400 2    50   BiDi ~ 0
 D7
@@
 Connection ~ 7000 2600
 Wire Wire Line
-	7350 2700 6850 2700
-Wire Wire Line
-	6850 5400 7450 5400
-Wire Wire Line
 	4500 4100 4500 6800
 Connection ~ 4500 4100
 Wire Wire Line
 	7350 3000 6850 3000
-Text HLabel 6850 6300 2    50   Input ~ 0
-~BLE
-Text Notes 7950 3200 0    197  ~ 0
+Text Notes 7950 2150 0    197  ~ 0
 High Bank
-Text Notes 7950 5700 0    197  ~ 0
+Text Notes 8050 7450 0    197  ~ 0
 Low Bank
-Text HLabel 7350 2700 2    50   Input ~ 0
+Text HLabel 6850 2700 2    50   Input ~ 0
 WE
-Text HLabel 7450 5400 2    50   Input ~ 0
+Text HLabel 6850 5400 2    50   Input ~ 0
 WE
-Text HLabel 6850 3600 2    50   Input ~ 0
-~BHE
 Text HLabel 6850 3400 2    50   Input ~ 0
 ~OE
@@
 	0    -1   -1   0
 $EndComp
+Text Notes 3500 7950 0    118  ~ 0
+Address Range: DFFFFh - FFFFFh (917503 - 1048575 dec)
+Wire Wire Line
+	6850 6300 8500 6300
+Wire Wire Line
+	6850 3600 8500 3600
+$Comp
+L Logic_Programmable:PAL16L8 U?
+U 1 1 5EA7EE08
+P 10350 4550
+F 0 "U?" H 10350 5431 50  0000 C CNN
+F 1 "PAL16L8" H 10350 5340 50  0000 C CNN
+F 2 "" H 10350 4550 50  0001 C CNN
+F 3 "" H 10350 4550 50  0001 C CNN
+	1    10350 4550
+	1    0    0    -1
+$EndComp
+Text HLabel 10850 4050 2    50   Input ~ 0
+A19
+Text HLabel 10850 4150 2    50   Input ~ 0
+A18
+Text HLabel 10850 4250 2    50   Input ~ 0
+A17
+Text HLabel 10850 4350 2    50   Input ~ 0
+~BLE
+Text HLabel 10850 4450 2    50   Input ~ 0
+~BHE
+Wire Wire Line
+	9850 4050 8500 4050
+Wire Wire Line
+	8500 4050 8500 3600
+Wire Wire Line
+	9850 4150 8500 4150
+Wire Wire Line
+	8500 4150 8500 6300
+Text HLabel 3600 6400 0    50   Input ~ 0
+~BHE
+Text HLabel 3600 6300 0    50   Input ~ 0
+A1
+Text HLabel 3600 6200 0    50   Input ~ 0
+A2
+Text HLabel 3600 6100 0    50   Input ~ 0
+A3
+Text HLabel 3600 6000 0    50   Input ~ 0
+A4
+Text HLabel 3600 5900 0    50   Input ~ 0
+A5
+Text HLabel 3600 5800 0    50   Input ~ 0
+A6
+Text HLabel 3600 5700 0    50   Input ~ 0
+A7
+Text HLabel 7350 5800 2    50   Input ~ 0
+A8
+Text HLabel 7350 5900 2    50   Input ~ 0
+A9
+Text HLabel 7350 6200 2    50   Input ~ 0
+A10
+Text HLabel 7350 6000 2    50   Input ~ 0
+A11
+Text HLabel 3600 5600 0    50   Input ~ 0
+A12
+Text HLabel 7350 5700 2    50   Input ~ 0
+A13
+Text HLabel 7350 5600 2    50   Input ~ 0
+A14
+Text HLabel 3600 5500 0    50   Input ~ 0
+A15
+Text HLabel 3600 5400 0    50   Input ~ 0
+A16
+Text HLabel 3600 3700 0    50   Input ~ 0
+~BHE
+Text HLabel 3600 3600 0    50   Input ~ 0
+A1
+Text HLabel 3600 3500 0    50   Input ~ 0
+A2
+Text HLabel 3600 3400 0    50   Input ~ 0
+A3
+Text HLabel 3600 3300 0    50   Input ~ 0
+A4
+Text HLabel 3600 3200 0    50   Input ~ 0
+A5
+Text HLabel 3600 3100 0    50   Input ~ 0
+A6
+Text HLabel 3600 3000 0    50   Input ~ 0
+A7
+Text HLabel 3600 2900 0    50   Input ~ 0
+A12
+Text HLabel 3600 2800 0    50   Input ~ 0
+A15
+Text HLabel 3600 2700 0    50   Input ~ 0
+A16
+Text HLabel 7350 3100 2    50   Input ~ 0
+A8
+Text HLabel 7350 3200 2    50   Input ~ 0
+A9
+Text HLabel 7350 3500 2    50   Input ~ 0
+A10
+Text HLabel 7350 3300 2    50   Input ~ 0
+A11
+Text HLabel 7350 3000 2    50   Input ~ 0
+A13
+Text HLabel 7350 2900 2    50   Input ~ 0
+A14
 $EndSCHEMATC
