File: Proj_5/Clock_Generator.sch (KiCad schematic (older format))
At the start: 5 parts

Commit message: Added at least 4 Footprints
Parts:
- C2: footprint (none) -> Capacitor_Tantalum_SMD:CP_EIA-1608-08_AVX-J
- CLK_R1, CLK_R2: footprint (none) -> Resistor_SMD:R_0201_0603Metric
- OSC1: footprint (none) -> Oscillator:Oscillator_DIP-8
Changed lines of the file:
@@
 F 0 "OSC1" V 3904 3081 50  0000 L CNN
 F 1 "24 MHz Crystal OSC" V 3995 3081 50  0000 L CNN
-F 2 "" H 3950 2950 50  0001 C CNN
+F 2 "Oscillator:Oscillator_DIP-8" H 3950 2950 50  0001 C CNN
 F 3 "~" H 3950 2950 50  0001 C CNN
 	1    3950 2950
@@
 F 0 "CLK_R1" V 4193 2800 50  0000 C CNN
 F 1 "510 Ohm" V 4284 2800 50  0000 C CNN
-F 2 "" V 4330 2800 50  0001 C CNN
+F 2 "Resistor_SMD:R_0201_0603Metric" V 4330 2800 50  0001 C CNN
 F 3 "~" H 4400 2800 50  0001 C CNN
 	1    4400 2800
@@
 F 0 "CLK_R2" V 4193 3350 50  0000 C CNN
 F 1 "510 Ohm" V 4284 3350 50  0000 C CNN
-F 2 "" V 4330 3350 50  0001 C CNN
+F 2 "Resistor_SMD:R_0201_0603Metric" V 4330 3350 50  0001 C CNN
 F 3 "~" H 4400 3350 50  0001 C CNN
 	1    4400 3350
@@
 F 0 "C2" V 1898 1250 50  0000 C CNN
 F 1 "0.1uF" V 1989 1250 50  0000 C CNN
-F 2 "" H 2188 1100 50  0001 C CNN
+F 2 "Capacitor_Tantalum_SMD:CP_EIA-1608-08_AVX-J" H 2188 1100 50  0001 C CNN
 F 3 "~" H 2150 1250 50  0001 C CNN
 	1    2150 1250

Commit message: Scary
Parts:
- OSC1: footprint Oscillator:Oscillator_DIP-8 -> Crystal:Crystal_DS10_D1.0mm_L4.3mm_Horizontal
Changed lines of the file:
@@
 F 0 "OSC1" V 3904 3081 50  0000 L CNN
 F 1 "24 MHz Crystal OSC" V 3995 3081 50  0000 L CNN
-F 2 "Oscillator:Oscillator_DIP-8" H 3950 2950 50  0001 C CNN
+F 2 "Crystal:Crystal_DS10_D1.0mm_L4.3mm_Horizontal" H 3950 2950 50  0001 C CNN
 F 3 "~" H 3950 2950 50  0001 C CNN
 	1    3950 2950

Commit message: Fixed 'Pad too close to Pad' Errors
Parts:
- CLK_R1, CLK_R2: footprint Resistor_SMD:R_0201_0603Metric -> Resistor_SMD:R_1206_3216Metric
Changed lines of the file:
@@
 F 0 "CLK_R1" V 4193 2800 50  0000 C CNN
 F 1 "510 Ohm" V 4284 2800 50  0000 C CNN
-F 2 "Resistor_SMD:R_0201_0603Metric" V 4330 2800 50  0001 C CNN
+F 2 "Resistor_SMD:R_1206_3216Metric" V 4330 2800 50  0001 C CNN
 F 3 "~" H 4400 2800 50  0001 C CNN
 	1    4400 2800
@@
 F 0 "CLK_R2" V 4193 3350 50  0000 C CNN
 F 1 "510 Ohm" V 4284 3350 50  0000 C CNN
-F 2 "Resistor_SMD:R_0201_0603Metric" V 4330 3350 50  0001 C CNN
+F 2 "Resistor_SMD:R_1206_3216Metric" V 4330 3350 50  0001 C CNN
 F 3 "~" H 4400 3350 50  0001 C CNN
 	1    4400 3350
