File: Proj_5/CY7C199.sch (KiCad schematic (older format))
At the start: 0 parts

Commit message: Added Caps to Each Vcc per desc.
Parts:
- added C? (x4): 0.1uF, symbol Device:C
- added U? (x4): CY7C199, symbol Memory_RAM:CY7C199
Connections:
- net labels added: GND
- wire segments 0 -> 12
Changed lines of the file:
@@
 Comment4 ""
 $EndDescr
+$Comp
+L Memory_RAM:CY7C199 U?
+U 1 1 5EA4313E
+P 4650 4500
+F 0 "U?" H 4650 5881 50  0000 C CNN
+F 1 "CY7C199" H 4650 5790 50  0000 C CNN
+F 2 "" H 4650 4500 50  0001 C CNN
+F 3 "" H 4650 4500 50  0001 C CNN
+	1    4650 4500
+	1    0    0    -1
+$EndComp
+$Comp
+L Memory_RAM:CY7C199 U?
+U 1 1 5EA4B54C
+P 7550 4500
+F 0 "U?" H 7550 5881 50  0000 C CNN
+F 1 "CY7C199" H 7550 5790 50  0000 C CNN
+F 2 "" H 7550 4500 50  0001 C CNN
+F 3 "" H 7550 4500 50  0001 C CNN
+	1    7550 4500
+	1    0    0    -1
+$EndComp
+$Comp
+L Memory_RAM:CY7C199 U?
+U 1 1 5EA4FA2E
+P 10850 4550
+F 0 "U?" H 10850 5931 50  0000 C CNN
+F 1 "CY7C199" H 10850 5840 50  0000 C CNN
+F 2 "" H 10850 4550 50  0001 C CNN
+F 3 "" H 10850 4550 50  0001 C CNN
+	1    10850 4550
+	1    0    0    -1
+$EndComp
+$Comp
+L Memory_RAM:CY7C199 U?
+U 1 1 5EA4FA34
+P 13750 4550
+F 0 "U?" H 13750 5931 50  0000 C CNN
+F 1 "CY7C199" H 13750 5840 50  0000 C CNN
+F 2 "" H 13750 4550 50  0001 C CNN
+F 3 "" H 13750 4550 50  0001 C CNN
+	1    13750 4550
+	1    0    0    -1
+$EndComp
+$Comp
+L Device:C C?
+U 1 1 5EA524F8
+P 14000 2900
+F 0 "C?" V 13748 2900 50  0000 C CNN
+F 1 "0.1uF" V 13839 2900 50  0000 C CNN
+F 2 "" H 14038 2750 50  0001 C CNN
+F 3 "~" H 14000 2900 50  0001 C CNN
+	1    14000 2900
+	0    1    1    0
+$EndComp
+$Comp
+L Device:C C?
+U 1 1 5EA53D82
+P 11100 2900
+F 0 "C?" V 10848 2900 50  0000 C CNN
+F 1 "0.1uF" V 10939 2900 50  0000 C CNN
+F 2 "" H 11138 2750 50  0001 C CNN
+F 3 "~" H 11100 2900 50  0001 C CNN
+	1    11100 2900
+	0    1    1    0
+$EndComp
+Wire Wire Line
+	13850 2900 13750 2900
+Wire Wire Line
+	13750 2900 13750 3350
+Wire Wire Line
+	13750 2900 13750 2600
+Connection ~ 13750 2900
+$Comp
+L power:GND #PWR?
+U 1 1 5EAA219F
+P 14150 2900
+AR Path="/5E9F3A3D/5EAA219F" Ref="#PWR?"  Part="1"
+AR Path="/5EA98353/5EAA219F" Ref="#PWR?"  Part="1"
+F 0 "#PWR?" H 14150 2650 50  0001 C CNN
+F 1 "GND" H 14155 2727 50  0000 C CNN
+F 2 "" H 14150 2900 50  0001 C CNN
+F 3 "" H 14150 2900 50  0001 C CNN
+	1    14150 2900
+	0    -1   -1   0
+$EndComp
+$Comp
+L power:GND #PWR?
+U 1 1 5EAA2618
+P 11250 2900
+AR Path="/5E9F3A3D/5EAA2618" Ref="#PWR?"  Part="1"
+AR Path="/5EA98353/5EAA2618" Ref="#PWR?"  Part="1"
+F 0 "#PWR?" H 11250 2650 50  0001 C CNN
+F 1 "GND" H 11255 2727 50  0000 C CNN
+F 2 "" H 11250 2900 50  0001 C CNN
+F 3 "" H 11250 2900 50  0001 C CNN
+	1    11250 2900
+	0    -1   -1   0
+$EndComp
+Wire Wire Line
+	10950 2900 10850 2900
+Wire Wire Line
+	10850 2900 10850 3350
+$Comp
+L Device:C C?
+U 1 1 5EAB250B
+P 7800 2850
+F 0 "C?" V 7548 2850 50  0000 C CNN
+F 1 "0.1uF" V 7639 2850 50  0000 C CNN
+F 2 "" H 7838 2700 50  0001 C CNN
+F 3 "~" H 7800 2850 50  0001 C CNN
+	1    7800 2850
+	0    1    1    0
+$EndComp
+Wire Wire Line
+	7650 2850 7550 2850
+Wire Wire Line
+	7550 2850 7550 3300
+Wire Wire Line
+	7550 2850 7550 2550
+Connection ~ 7550 2850
+$Comp
+L power:GND #PWR?
+U 1 1 5EAB2515
+P 7950 2850
+AR Path="/5E9F3A3D/5EAB2515" Ref="#PWR?"  Part="1"
+AR Path="/5EA98353/5EAB2515" Ref="#PWR?"  Part="1"
+F 0 "#PWR?" H 7950 2600 50  0001 C CNN
+F 1 "GND" H 7955 2677 50  0000 C CNN
+F 2 "" H 7950 2850 50  0001 C CNN
+F 3 "" H 7950 2850 50  0001 C CNN
+	1    7950 2850
+	0    -1   -1   0
+$EndComp
+$Comp
+L Device:C C?
+U 1 1 5EAB3F01
+P 4900 2850
+F 0 "C?" V 4648 2850 50  0000 C CNN
+F 1 "0.1uF" V 4739 2850 50  0000 C CNN
+F 2 "" H 4938 2700 50  0001 C CNN
+F 3 "~" H 4900 2850 50  0001 C CNN
+	1    4900 2850
+	0    1    1    0
+$EndComp
+Wire Wire Line
+	4750 2850 4650 2850
+Wire Wire Line
+	4650 2850 4650 3300
+Wire Wire Line
+	4650 2850 4650 2550
+Connection ~ 4650 2850
+$Comp
+L power:GND #PWR?
+U 1 1 5EAB3F0B
+P 5050 2850
+AR Path="/5E9F3A3D/5EAB3F0B" Ref="#PWR?"  Part="1"
+AR Path="/5EA98353/5EAB3F0B" Ref="#PWR?"  Part="1"
+F 0 "#PWR?" H 5050 2600 50  0001 C CNN
+F 1 "GND" H 5055 2677 50  0000 C CNN
+F 2 "" H 5050 2850 50  0001 C CNN
+F 3 "" H 5050 2850 50  0001 C CNN
+	1    5050 2850
+	0    -1   -1   0
+$EndComp
+Wire Wire Line
+	10850 2900 10850 2500
+Connection ~ 10850 2900
+$Comp
+L power:GND #PWR?
+U 1 1 5EAB5C11
+P 10850 5750
+AR Path="/5E9F3A3D/5EAB5C11" Ref="#PWR?"  Part="1"
+AR Path="/5EA98353/5EAB5C11" Ref="#PWR?"  Part="1"
+F 0 "#PWR?" H 10850 5500 50  0001 C CNN
+F 1 "GND" H 10855 5577 50  0000 C CNN
+F 2 "" H 10850 5750 50  0001 C CNN
+F 3 "" H 10850 5750 50  0001 C CNN
+	1    10850 5750
+	1    0    0    -1
+$EndComp
+$Comp
+L power:GND #PWR?
+U 1 1 5EAB5EF1
+P 13750 5750
+AR Path="/5E9F3A3D/5EAB5EF1" Ref="#PWR?"  Part="1"
+AR Path="/5EA98353/5EAB5EF1" Ref="#PWR?"  Part="1"
+F 0 "#PWR?" H 13750 5500 50  0001 C CNN
+F 1 "GND" H 13755 5577 50  0000 C CNN
+F 2 "" H 13750 5750 50  0001 C CNN
+F 3 "" H 13750 5750 50  0001 C CNN
+	1    13750 5750
+	1    0    0    -1
+$EndComp
+$Comp
+L power:GND #PWR?
+U 1 1 5EAB6217
+P 7550 5700
+AR Path="/5E9F3A3D/5EAB6217" Ref="#PWR?"  Part="1"
+AR Path="/5EA98353/5EAB6217" Ref="#PWR?"  Part="1"
+F 0 "#PWR?" H 7550 5450 50  0001 C CNN
+F 1 "GND" H 7555 5527 50  0000 C CNN
+F 2 "" H 7550 5700 50  0001 C CNN
+F 3 "" H 7550 5700 50  0001 C CNN
+	1    7550 5700
+	1    0    0    -1
+$EndComp
+$Comp
+L power:GND #PWR?
+U 1 1 5EAB6544
+P 4650 5700
+AR Path="/5E9F3A3D/5EAB6544" Ref="#PWR?"  Part="1"
+AR Path="/5EA98353/5EAB6544" Ref="#PWR?"  Part="1"
+F 0 "#PWR?" H 4650 5450 50  0001 C CNN
+F 1 "GND" H 4655 5527 50  0000 C CNN
+F 2 "" H 4650 5700 50  0001 C CNN
+F 3 "" H 4650 5700 50  0001 C CNN
+	1    4650 5700
+	1    0    0    -1
+$EndComp
 $EndSCHEMATC
