File: Proj_5/CY7C199.sch (KiCad schematic (older format))
At the start: 10 parts, among them U5 CY7C199, U6 CY7C199, U7 PAL16L8, U8 CY7C199, U9 CY7C199

Commit message: Added at least 4 Footprints
Parts:
- C1, C3, C4, C5, C6: footprint (none) -> Capacitor_Tantalum_SMD:CP_EIA-1608-08_AVX-J
- U5, U6, U8, U9: footprint (none) -> Package_DIP:DIP-28_W15.24mm
- U7: footprint (none) -> Package_DIP:DIP-20_W7.62mm
Changed lines of the file:
@@
 F 0 "U5" H 5400 7981 50  0000 C CNN
 F 1 "CY7C199" H 5400 7890 50  0000 C CNN
-F 2 "" H 5400 6600 50  0001 C CNN
+F 2 "Package_DIP:DIP-28_W15.24mm" H 5400 6600 50  0001 C CNN
 F 3 "" H 5400 6600 50  0001 C CNN
 	1    5400 6600
@@
 F 0 "U6" H 5400 11581 50  0000 C CNN
 F 1 "CY7C199" H 5400 11490 50  0000 C CNN
-F 2 "" H 5400 10200 50  0001 C CNN
+F 2 "Package_DIP:DIP-28_W15.24mm" H 5400 10200 50  0001 C CNN
 F 3 "" H 5400 10200 50  0001 C CNN
 	1    5400 10200
@@
 F 0 "U8" H 10450 7981 50  0000 C CNN
 F 1 "CY7C199" H 10450 7890 50  0000 C CNN
-F 2 "" H 10450 6600 50  0001 C CNN
+F 2 "Package_DIP:DIP-28_W15.24mm" H 10450 6600 50  0001 C CNN
 F 3 "" H 10450 6600 50  0001 C CNN
 	1    10450 6600
@@
 F 0 "U9" H 10450 11581 50  0000 C CNN
 F 1 "CY7C199" H 10450 11490 50  0000 C CNN
-F 2 "" H 10450 10200 50  0001 C CNN
+F 2 "Package_DIP:DIP-28_W15.24mm" H 10450 10200 50  0001 C CNN
 F 3 "" H 10450 10200 50  0001 C CNN
 	1    10450 10200
@@
 F 0 "U7" H 5750 4481 50  0000 C CNN
 F 1 "PAL16L8" H 5750 4390 50  0000 C CNN
-F 2 "" H 5750 3600 50  0001 C CNN
+F 2 "Package_DIP:DIP-20_W7.62mm" H 5750 3600 50  0001 C CNN
 F 3 "" H 5750 3600 50  0001 C CNN
 	1    5750 3600
@@
 F 0 "C4" V 7498 3600 50  0000 C CNN
 F 1 "0.1uF" V 7589 3600 50  0000 C CNN
-F 2 "" H 7788 3450 50  0001 C CNN
+F 2 "Capacitor_Tantalum_SMD:CP_EIA-1608-08_AVX-J" H 7788 3450 50  0001 C CNN
 F 3 "~" H 7750 3600 50  0001 C CNN
 	1    7750 3600
@@
 F 0 "C1" V 4848 5150 50  0000 C CNN
 F 1 "0.1uF" V 4939 5150 50  0000 C CNN
-F 2 "" H 5138 5000 50  0001 C CNN
+F 2 "Capacitor_Tantalum_SMD:CP_EIA-1608-08_AVX-J" H 5138 5000 50  0001 C CNN
 F 3 "~" H 5100 5150 50  0001 C CNN
 	1    5100 5150
@@
 F 0 "C3" V 4898 8750 50  0000 C CNN
 F 1 "0.1uF" V 4989 8750 50  0000 C CNN
-F 2 "" H 5188 8600 50  0001 C CNN
+F 2 "Capacitor_Tantalum_SMD:CP_EIA-1608-08_AVX-J" H 5188 8600 50  0001 C CNN
 F 3 "~" H 5150 8750 50  0001 C CNN
 	1    5150 8750
@@
 F 0 "C5" V 9948 5150 50  0000 C CNN
 F 1 "0.1uF" V 10039 5150 50  0000 C CNN
-F 2 "" H 10238 5000 50  0001 C CNN
+F 2 "Capacitor_Tantalum_SMD:CP_EIA-1608-08_AVX-J" H 10238 5000 50  0001 C CNN
 F 3 "~" H 10200 5150 50  0001 C CNN
 	1    10200 5150
@@
 F 0 "C6" V 9998 8750 50  0000 C CNN
 F 1 "0.1uF" V 10089 8750 50  0000 C CNN
-F 2 "" H 10288 8600 50  0001 C CNN
+F 2 "Capacitor_Tantalum_SMD:CP_EIA-1608-08_AVX-J" H 10288 8600 50  0001 C CNN
 F 3 "~" H 10250 8750 50  0001 C CNN
 	1    10250 8750

Commit message: Data Aquired
Connections:
- net D0: no longer U8.11 (D0), U9.11 (D0)
- net D1: no longer U8.12 (D1), U9.12 (D1)
- net D2: no longer U8.13 (D2), U9.13 (D2)
- net D3: no longer U8.15 (D3), U9.15 (D3)
- net D4: no longer U8.16 (D4), U9.16 (D4)
- net D5: no longer U8.17 (D5), U9.17 (D5)
- net D6: no longer U8.18 (D6), U9.18 (D6)
- net D7: no longer U8.19 (D7), U9.19 (D7)
- new net D10: U8.13 (D2), U9.13 (D2)
- new net D11: U8.15 (D3), U9.15 (D3)
- new net D12: U8.16 (D4), U9.16 (D4)
- new net D13: U8.17 (D5), U9.17 (D5)
- new net D14: U8.18 (D6), U9.18 (D6)
- new net D15: U8.19 (D7), U9.19 (D7)
- new net D8: U8.11 (D0), U9.11 (D0)
- new net D9: U8.12 (D1), U9.12 (D1)

Commit message: Wires are Hell
Parts:
- removed C4: 0.1uF, Capacitor_Tantalum_SMD:CP_EIA-1608-08_AVX-J, symbol Device:C
Changed lines of the file:
@@
 	1    0    0    -1
 $EndComp
-$Comp
-L Device:C C4
-U 1 1 5F0B1B35
-P 7750 3600
-AR Path="/5EA98353/5F0B1B35" Ref="C4"  Part="1"
-AR Path="/5EA98A67/5F0B1B35" Ref="C?"  Part="1"
-AR Path="/5EC03876/5F0B1B35" Ref="C?"  Part="1"
-AR Path="/5ED6EB57/5F0B1B35" Ref="C?"  Part="1"
-F 0 "C4" V 7498 3600 50  0000 C CNN
-F 1 "0.1uF" V 7589 3600 50  0000 C CNN
-F 2 "Capacitor_Tantalum_SMD:CP_EIA-1608-08_AVX-J" H 7788 3450 50  0001 C CNN
-F 3 "~" H 7750 3600 50  0001 C CNN
-	1    7750 3600
-	0    1    1    0
-$EndComp
-$Comp
-L power:GND #PWR?
-U 1 1 5F0B1B3B
-P 7900 3600
-AR Path="/5EAF7226/5F0B1B3B" Ref="#PWR?"  Part="1"
-AR Path="/5EA98A67/5F0B1B3B" Ref="#PWR?"  Part="1"
-AR Path="/5EA98353/5F0B1B3B" Ref="#PWR015"  Part="1"
-AR Path="/5EC03876/5F0B1B3B" Ref="#PWR?"  Part="1"
-AR Path="/5ED6EB57/5F0B1B3B" Ref="#PWR?"  Part="1"
-F 0 "#PWR015" H 7900 3350 50  0001 C CNN
-F 1 "GND" H 7905 3427 50  0000 C CNN
-F 2 "" H 7900 3600 50  0001 C CNN
-F 3 "" H 7900 3600 50  0001 C CNN
-	1    7900 3600
-	0    -1   -1   0
-$EndComp
-Wire Wire Line
-	7600 3600 7150 3600
 Wire Wire Line
 	7150 3250 7150 3600
-Connection ~ 7150 3600
 Wire Wire Line
 	7150 3600 6450 3600
