File: Proj_5/16550UART.sch (KiCad schematic (older format))
At the start: 10 parts, among them J7 DSUB-9, U14 16550, U51 PAL16L8, U52 74AHC1G02, U53 74LVC1G08, U54 74AHC1G02, U55 max235cpg

Commit message: Power Flags
Connections:
- net GND: now also U55.20 (*EN); no longer U55.21 (SHDN)
- net VCC: no longer U55.20 (*EN)
- no-connect marks 31 -> 32
Changed lines of the file:
@@
 NoConn ~ 5900 6850
 NoConn ~ 5900 6950
-$Comp
-L power:GND #PWR0105
-U 1 1 5EAB604F
-P 16650 7000
-F 0 "#PWR0105" H 16650 6750 50  0001 C CNN
-F 1 "GND" V 16655 6872 50  0000 R CNN
-F 2 "" H 16650 7000 50  0001 C CNN
-F 3 "" H 16650 7000 50  0001 C CNN
-	1    16650 7000
-	0    -1   -1   0
-$EndComp
-$Comp
-L power:VCC #PWR097
-U 1 1 5EAB6B80
-P 14050 7000
-F 0 "#PWR097" H 14050 6850 50  0001 C CNN
-F 1 "VCC" H 14067 7173 50  0000 C CNN
-F 2 "" H 14050 7000 50  0001 C CNN
-F 3 "" H 14050 7000 50  0001 C CNN
-	1    14050 7000
-	1    0    0    -1
-$EndComp
 Wire Wire Line
 	9200 5200 9200 5650
@@
 Text HLabel 8200 6900 0    50   BiDi ~ 0
 D15
-$Comp
-L power:PWR_FLAG #FLG?
-U 1 1 5EDA95FE
-P 7400 7400
-F 0 "#FLG?" H 7400 7475 50  0001 C CNN
-F 1 "PWR_FLAG" V 7400 7527 50  0000 L CNN
-F 2 "" H 7400 7400 50  0001 C CNN
-F 3 "~" H 7400 7400 50  0001 C CNN
-	1    7400 7400
-	0    -1   -1   0
-$EndComp
-Connection ~ 7400 7400
 Wire Wire Line
 	5400 6550 5200 6550
@@
 	5400 7850 5400 8000
 $Comp
-L power:VCC #PWR?
+L power:VCC #PWR029
 U 1 1 5EDADCA7
 P 5200 6300
-F 0 "#PWR?" H 5200 6150 50  0001 C CNN
+F 0 "#PWR029" H 5200 6150 50  0001 C CNN
 F 1 "VCC" H 5217 6473 50  0000 C CNN
 F 2 "" H 5200 6300 50  0001 C CNN
@@
 P 5400 8000
 AR Path="/5EAF7226/5EDB05EC" Ref="#PWR?"  Part="1"
-AR Path="/5EA98A67/5EDB05EC" Ref="#PWR?"  Part="1"
-F 0 "#PWR?" H 5400 7750 50  0001 C CNN
+AR Path="/5EA98A67/5EDB05EC" Ref="#PWR030"  Part="1"
+F 0 "#PWR030" H 5400 7750 50  0001 C CNN
 F 1 "GND" H 5405 7827 50  0000 C CNN
 F 2 "" H 5400 8000 50  0001 C CNN
@@
 $EndComp
 $Comp
-L power:PWR_FLAG #FLG?
-U 1 1 5EDB2807
-P 5400 8000
-F 0 "#FLG?" H 5400 8075 50  0001 C CNN
-F 1 "PWR_FLAG" V 5400 8127 50  0000 L CNN
-F 2 "" H 5400 8000 50  0001 C CNN
-F 3 "~" H 5400 8000 50  0001 C CNN
-	1    5400 8000
-	0    -1   -1   0
-$EndComp
-$Comp
-L power:PWR_FLAG #FLG?
-U 1 1 5EDB3E22
-P 9200 5200
-F 0 "#FLG?" H 9200 5275 50  0001 C CNN
-F 1 "PWR_FLAG" V 9200 5327 50  0000 L CNN
-F 2 "" H 9200 5200 50  0001 C CNN
-F 3 "~" H 9200 5200 50  0001 C CNN
-	1    9200 5200
-	0    1    1    0
-$EndComp
-Connection ~ 9200 5200
-Connection ~ 5400 8000
-$Comp
-L power:PWR_FLAG #FLG?
-U 1 1 5EDB8A2E
-P 5200 6300
-F 0 "#FLG?" H 5200 6375 50  0001 C CNN
-F 1 "PWR_FLAG" V 5200 6427 50  0000 L CNN
-F 2 "" H 5200 6300 50  0001 C CNN
-F 3 "~" H 5200 6300 50  0001 C CNN
-	1    5200 6300
-	0    -1   -1   0
-$EndComp
-$Comp
-L power:PWR_FLAG #FLG?
-U 1 1 5EDBA7F8
-P 9200 9300
-F 0 "#FLG?" H 9200 9375 50  0001 C CNN
-F 1 "PWR_FLAG" V 9200 9427 50  0000 L CNN
-F 2 "" H 9200 9300 50  0001 C CNN
-F 3 "~" H 9200 9300 50  0001 C CNN
-	1    9200 9300
-	0    1    1    0
-$EndComp
-$Comp
-L power:VCC #PWR?
+L power:VCC #PWR031
 U 1 1 5EDC0795
 P 15700 9600
-F 0 "#PWR?" H 15700 9450 50  0001 C CNN
+F 0 "#PWR031" H 15700 9450 50  0001 C CNN
 F 1 "VCC" H 15717 9773 50  0000 C CNN
 F 2 "" H 15700 9600 50  0001 C CNN
@@
 	-1   0    0    1
 $EndComp
-$Comp
-L power:PWR_FLAG #FLG?
-U 1 1 5EDC079B
-P 15700 9600
-F 0 "#FLG?" H 15700 9675 50  0001 C CNN
-F 1 "PWR_FLAG" V 15700 9727 50  0000 L CNN
-F 2 "" H 15700 9600 50  0001 C CNN
-F 3 "~" H 15700 9600 50  0001 C CNN
-	1    15700 9600
-	0    -1   -1   0
-$EndComp
-Connection ~ 15700 9600
 Wire Wire Line
 	15700 8600 15700 9600
 $Comp
-L power:PWR_FLAG #FLG?
-U 1 1 5EDC2E00
-P 19550 8200
-F 0 "#FLG?" H 19550 8275 50  0001 C CNN
-F 1 "PWR_FLAG" V 19550 8327 50  0000 L CNN
-F 2 "" H 19550 8200 50  0001 C CNN
-F 3 "~" H 19550 8200 50  0001 C CNN
-	1    19550 8200
-	0    -1   -1   0
+L power:GND #PWR?
+U 1 1 5F37E591
+P 14050 7000
+F 0 "#PWR?" H 14050 6750 50  0001 C CNN
+F 1 "GND" V 14055 6872 50  0000 R CNN
+F 2 "" H 14050 7000 50  0001 C CNN
+F 3 "" H 14050 7000 50  0001 C CNN
+	1    14050 7000
+	0    1    1    0
 $EndComp
-$Comp
-L power:PWR_FLAG #FLG?
-U 1 1 5EDC65AB
-P 15000 8600
-F 0 "#FLG?" H 15000 8675 50  0001 C CNN
-F 1 "PWR_FLAG" V 15000 8727 50  0000 L CNN
-F 2 "" H 15000 8600 50  0001 C CNN
-F 3 "~" H 15000 8600 50  0001 C CNN
-	1    15000 8600
-	0    -1   -1   0
-$EndComp
-$Comp
-L power:PWR_FLAG #FLG?
-U 1 1 5EDC8FD2
-P 16650 7000
-F 0 "#FLG?" H 16650 7075 50  0001 C CNN
-F 1 "PWR_FLAG" V 16650 7127 50  0000 L CNN
-F 2 "" H 16650 7000 50  0001 C CNN
-F 3 "~" H 16650 7000 50  0001 C CNN
-	1    16650 7000
-	1    0    0    -1
-$EndComp
-$Comp
-L power:PWR_FLAG #FLG?
-U 1 1 5EDCA580
-P 14050 7000
-F 0 "#FLG?" H 14050 7075 50  0001 C CNN
-F 1 "PWR_FLAG" V 14050 7127 50  0000 L CNN
-F 2 "" H 14050 7000 50  0001 C CNN
-F 3 "~" H 14050 7000 50  0001 C CNN
-	1    14050 7000
-	0    -1   -1   0
-$EndComp
+NoConn ~ 16650 7000
 $EndSCHEMATC
