File: Proj_5/Display_LEDS.sch (KiCad schematic (older format))
At the start: 10 parts, among them U15 74LVC1G11, U16 74LVC1G11, U26 74LVC1G11, U27 74LVC1G11, U28 74LVC1G11, U29 74LVC1G11, U30 74LVC1G11, U31 74LVC1G11, U32 PAL16L8

Commit message: 11 errors left
Connections:
- no-connect marks 0 -> 17
Changed lines of the file:
@@
 $Descr A2 23386 16535
 encoding utf-8
-Sheet 10 10
+Sheet 9 10
 Title ""
 Date ""
@@
 RS
 $Comp
-L power:+3V0 #PWR027
-U 1 1 5EBB715E
-P 12600 2500
-F 0 "#PWR027" H 12600 2350 50  0001 C CNN
-F 1 "+3V0" V 12615 2628 50  0000 L CNN
-F 2 "" H 12600 2500 50  0001 C CNN
-F 3 "" H 12600 2500 50  0001 C CNN
-	1    12600 2500
-	0    1    1    0
-$EndComp
-$Comp
 L power:GND #PWR028
 U 1 1 5EBB7839
@@
 $EndComp
 $Comp
-L power:+3.3V #PWR025
-U 1 1 5EBBD5A0
-P 11500 2200
-F 0 "#PWR025" H 11500 2050 50  0001 C CNN
-F 1 "+3.3V" V 11515 2328 50  0000 L CNN
-F 2 "" H 11500 2200 50  0001 C CNN
-F 3 "" H 11500 2200 50  0001 C CNN
-	1    11500 2200
-	0    -1   -1   0
-$EndComp
-$Comp
 L power:GND #PWR024
 U 1 1 5EBBE088
@@
 Wire Wire Line
 	8450 3200 8450 3350
+NoConn ~ 12600 2700
+NoConn ~ 12600 2800
+NoConn ~ 12600 2900
+NoConn ~ 12600 3000
+$Comp
+L power:+3V0 #PWR0129
+U 1 1 5EBC7EC9
+P 12800 2500
+F 0 "#PWR0129" H 12800 2350 50  0001 C CNN
+F 1 "+3V0" V 12815 2628 50  0000 L CNN
+F 2 "" H 12800 2500 50  0001 C CNN
+F 3 "" H 12800 2500 50  0001 C CNN
+	1    12800 2500
+	0    1    1    0
+$EndComp
+$Comp
+L power:+3V3 #PWR0130
+U 1 1 5EBC9461
+P 11300 2200
+F 0 "#PWR0130" H 11300 2050 50  0001 C CNN
+F 1 "+3V3" V 11315 2328 50  0000 L CNN
+F 2 "" H 11300 2200 50  0001 C CNN
+F 3 "" H 11300 2200 50  0001 C CNN
+	1    11300 2200
+	0    -1   -1   0
+$EndComp
+NoConn ~ 8950 2100
+NoConn ~ 8950 2200
+NoConn ~ 8950 2300
+NoConn ~ 8950 2400
+NoConn ~ 8950 2500
+NoConn ~ 8950 2600
+NoConn ~ 8950 2700
+NoConn ~ 7950 2500
+NoConn ~ 7950 2600
+NoConn ~ 7950 2700
+NoConn ~ 7950 2800
+NoConn ~ 7950 2900
+NoConn ~ 7950 3000
+Wire Wire Line
+	11300 2200 11500 2200
+Wire Wire Line
+	12800 2500 12600 2500
+Entry Wire Line
+	11350 15000 11250 14900
+Entry Wire Line
+	11450 15000 11350 14900
+Wire Wire Line
+	11250 14900 11250 14500
+Wire Wire Line
+	11350 14900 11350 14500
 Wire Bus Line
 	1500 600  12300 600
 Wire Bus Line
+	1500 600  1500 15000
+Wire Bus Line
 	1500 15000 12350 15000
-Wire Bus Line
-	1500 600  1500 15000
+Text HLabel 11250 14500 1    50   Input ~ 0
+R~W
+Text HLabel 11350 14500 1    50   Input ~ 0
+RS
+Text Label 11250 14900 1    50   ~ 0
+R~W
+Text Label 11350 14900 1    50   ~ 0
+RS
 $EndSCHEMATC

Commit message: 1 Error Remains
Connections:
- net +3V3 is gone; now on net VCC: DS1.2 (VDD)
- net GND: no longer DS1.16 (LED-)
- net RS: no longer DS1.4 (RS)
- net R~W: no longer DS1.5 (R/W)
- net at U32.13 (IO7): now also DS1.5 (R/W)
- net at U32.14 (IO6): now also DS1.4 (RS)
- net +3V0: no longer names the net of DS1.15 (LED+)
Changed lines of the file:
@@
 Wire Wire Line
 	11500 2600 9350 2600
-Wire Wire Line
-	11500 2500 10250 2500
-Wire Wire Line
-	10250 2500 10250 700
-Entry Wire Line
-	10150 600  10250 700
-Text Label 10250 850  1    50   ~ 0
-R~W
-Wire Wire Line
-	11500 2400 10350 2400
-Wire Wire Line
-	10350 2400 10350 700
-Entry Wire Line
-	10250 600  10350 700
-Text Label 10350 850  1    50   ~ 0
-RS
-$Comp
-L power:GND #PWR028
-U 1 1 5EBB7839
-P 12600 2600
-F 0 "#PWR028" H 12600 2350 50  0001 C CNN
-F 1 "GND" V 12605 2472 50  0000 R CNN
-F 2 "" H 12600 2600 50  0001 C CNN
-F 3 "" H 12600 2600 50  0001 C CNN
-	1    12600 2600
-	0    -1   -1   0
-$EndComp
 $Comp
 L power:GND #PWR026
@@
 NoConn ~ 12600 2900
 NoConn ~ 12600 3000
-$Comp
-L power:+3V0 #PWR0129
-U 1 1 5EBC7EC9
-P 12800 2500
-F 0 "#PWR0129" H 12800 2350 50  0001 C CNN
-F 1 "+3V0" V 12815 2628 50  0000 L CNN
-F 2 "" H 12800 2500 50  0001 C CNN
-F 3 "" H 12800 2500 50  0001 C CNN
-	1    12800 2500
-	0    1    1    0
-$EndComp
-$Comp
-L power:+3V3 #PWR0130
-U 1 1 5EBC9461
-P 11300 2200
-F 0 "#PWR0130" H 11300 2050 50  0001 C CNN
-F 1 "+3V3" V 11315 2328 50  0000 L CNN
-F 2 "" H 11300 2200 50  0001 C CNN
-F 3 "" H 11300 2200 50  0001 C CNN
-	1    11300 2200
-	0    -1   -1   0
-$EndComp
 NoConn ~ 8950 2100
 NoConn ~ 8950 2200
@@
 NoConn ~ 8950 2400
 NoConn ~ 8950 2500
-NoConn ~ 8950 2600
-NoConn ~ 8950 2700
 NoConn ~ 7950 2500
 NoConn ~ 7950 2600
@@
 Wire Wire Line
 	11300 2200 11500 2200
-Wire Wire Line
-	12800 2500 12600 2500
 Entry Wire Line
 	11350 15000 11250 14900
@@
 Wire Wire Line
 	11350 14900 11350 14500
-Wire Bus Line
-	1500 600  12300 600
-Wire Bus Line
-	1500 600  1500 15000
-Wire Bus Line
-	1500 15000 12350 15000
 Text HLabel 11250 14500 1    50   Input ~ 0
 R~W
@@
 Text Label 11350 14900 1    50   ~ 0
 RS
+$Comp
+L power:VCC #PWR0129
+U 1 1 5ED3DC79
+P 11300 2200
+F 0 "#PWR0129" H 11300 2050 50  0001 C CNN
+F 1 "VCC" H 11317 2373 50  0000 C CNN
+F 2 "" H 11300 2200 50  0001 C CNN
+F 3 "" H 11300 2200 50  0001 C CNN
+	1    11300 2200
+	0    -1   -1   0
+$EndComp
+NoConn ~ 12600 2500
+NoConn ~ 12600 2600
+Wire Wire Line
+	11500 2500 9300 2500
+Wire Wire Line
+	9300 2500 9300 2700
+Wire Wire Line
+	9300 2700 8950 2700
+Wire Wire Line
+	8950 2600 9250 2600
+Wire Wire Line
+	9250 2600 9250 2400
+Wire Wire Line
+	9250 2400 11500 2400
+Wire Bus Line
+	1500 600  12300 600
+Wire Bus Line
+	1500 600  1500 15000
+Wire Bus Line
+	1500 15000 12350 15000
 $EndSCHEMATC

Commit message: Added 5 Footprints
Parts:
- DS1: footprint LCD4x20 -> parts:LCD4x20
Changed lines of the file:
@@
 F 0 "DS1" H 12050 2365 50  0000 C CNN
 F 1 "LCD4x20" H 12050 2274 50  0000 C CNN
-F 2 "LCD4x20" H 12450 2200 50  0001 L CNN
+F 2 "parts:LCD4x20" H 12450 2200 50  0001 L CNN
 F 3 "https://componentsearchengine.com/Datasheets/1/LCD4x20.pdf" H 12450 2100 50  0001 L CNN
 F 4 "LCD Character Display Modules & Accessories STN-Y/G Transfl 77.5 x 47.0" H 12450 2000 50  0001 L CNN "Description"
