File: Proj_5/Display.sch (KiCad schematic (older format))
At the start: 10 parts, among them U15 74LVC1G11, U16 74LVC1G11, U26 74LVC1G11, U27 74LVC1G11, U28 74LVC1G11, U29 74LVC1G11, U30 74LVC1G11, U31 74LVC1G11, U32 PAL16L8

Commit message: No more gates 2
Parts:
- removed U15, U16, U26, U27, U28, U29, U30, U31: 74LVC1G11, symbol 74xGxx:74LVC1G11
- removed U32: PAL16L8, Package_DIP:DIP-20_W7.62mm, symbol Logic_Programmable:PAL16L8
- added U15, U16: PAL16L8, Package_DIP:DIP-20_W7.62mm, symbol Logic_Programmable:PAL16L8
Connections:
- net A0: now also U16.8 (I8)
- net A1: now also U16.7 (I7)
- net A10: now also U15.11 (I10)
- net A11: now also U15.9 (I9)
- net A12: now also U15.8 (I8)
- net A13: now also U15.7 (I7)
- net A14: now also U15.6 (I6)
- net A15: now also U15.5 (I5)
- net A16: now also U15.4 (I4)
- net A17: now also U15.3 (I3)
- net A18: now also U15.2 (I2)
- net A19: now also U15.1 (I1)
- net A2: now also U16.6 (I6)
- net A3: now also U16.5 (I5)
- net A4: now also U16.4 (I4)
- net A5: now also U16.3 (I3)
- net A6: now also U16.2 (I2)
- net A7: now also U16.1 (I1)
- net A8: now also U15.14 (IO6)
- net A9: now also U15.13 (IO7)
- net GND: now also U15.10 (GND), U16.10 (GND)
- net VCC: now also U15.20 (VCC), U16.20 (VCC)
- net at DS1.6 (E): now also U16.17 (I03)
- net at DS1.5 (R/W): now also U16.18 (IO2)
- net at DS1.4 (RS): now also U16.19 (IO1)
- new net: U15.12 (IO8), U16.9 (I9)

Commit message: Playing with PCB placements
Parts:
- added C22: 0.1uF, Capacitor_Tantalum_SMD:CP_EIA-1608-08_AVX-J, symbol Device:C
Connections:
- net GND: now also C22.2
- net VCC: now also C22.1
Changed lines of the file:
@@
 NoConn ~ 12600 2900
 NoConn ~ 12600 3000
-Wire Wire Line
-	11300 2200 11500 2200
 $Comp
 L power:VCC #PWR0129
 U 1 1 5ED3DC79
-P 11300 2200
-F 0 "#PWR0129" H 11300 2050 50  0001 C CNN
-F 1 "VCC" H 11317 2373 50  0000 C CNN
-F 2 "" H 11300 2200 50  0001 C CNN
-F 3 "" H 11300 2200 50  0001 C CNN
-	1    11300 2200
+P 10400 1650
+F 0 "#PWR0129" H 10400 1500 50  0001 C CNN
+F 1 "VCC" H 10417 1823 50  0000 C CNN
+F 2 "" H 10400 1650 50  0001 C CNN
+F 3 "" H 10400 1650 50  0001 C CNN
+	1    10400 1650
 	0    -1   -1   0
 $EndComp
@@
 Wire Wire Line
 	2900 6000 3200 6000
+$Comp
+L Device:C C?
+U 1 1 5ED6A742
+P 10500 1900
+AR Path="/5EA98353/5ED6A742" Ref="C?"  Part="1"
+AR Path="/5EA99146/5ED6A742" Ref="C?"  Part="1"
+AR Path="/5EA993EC/5ED6A742" Ref="C?"  Part="1"
+AR Path="/5EAF7226/5ED6A742" Ref="C22"  Part="1"
+F 0 "C22" V 10248 1900 50  0000 C CNN
+F 1 "0.1uF" V 10339 1900 50  0000 C CNN
+F 2 "Capacitor_Tantalum_SMD:CP_EIA-1608-08_AVX-J" H 10538 1750 50  0001 C CNN
+F 3 "~" H 10500 1900 50  0001 C CNN
+	1    10500 1900
+	1    0    0    -1
+$EndComp
+$Comp
+L power:GND #PWR?
+U 1 1 5ED6A748
+P 10500 2050
+AR Path="/5EA993EC/5ED6A748" Ref="#PWR?"  Part="1"
+AR Path="/5EAF7226/5ED6A748" Ref="#PWR049"  Part="1"
+F 0 "#PWR049" H 10500 1800 50  0001 C CNN
+F 1 "GND" H 10505 1877 50  0000 C CNN
+F 2 "" H 10500 2050 50  0001 C CNN
+F 3 "" H 10500 2050 50  0001 C CNN
+	1    10500 2050
+	1    0    0    -1
+$EndComp
+Wire Wire Line
+	10400 1650 10500 1650
+Wire Wire Line
+	10500 1650 10500 1750
+Wire Wire Line
+	10500 1650 10900 1650
+Wire Wire Line
+	10900 1650 10900 2200
+Wire Wire Line
+	10900 2200 11500 2200
+Connection ~ 10500 1650
 Wire Bus Line
 	1500 600  12300 600
