File: Proj_5/LED_Switch.sch (KiCad schematic (older format))
At the start: 33 parts

Commit message: Finished Most of power flags, power connector header, added hierachical pins to a few sheets.
Connections:
- net GND: now also U?.10 (GND), U?.10 (GND)
- net VCC: now also U?.20 (VCC), U?.20 (VCC)
Changed lines of the file:
@@
 $Descr A2 23386 16535
 encoding utf-8
-Sheet 10 10
+Sheet 9 10
 Title ""
 Date ""
@@
 	1    0    0    -1
 $EndComp
+$Comp
+L power:VCC #PWR?
+U 1 1 5EDD0804
+P 15900 4300
+AR Path="/5EAF7226/5EDD0804" Ref="#PWR?"  Part="1"
+AR Path="/5EB38D8D/5EDD0804" Ref="#PWR?"  Part="1"
+F 0 "#PWR?" H 15900 4150 50  0001 C CNN
+F 1 "VCC" H 15917 4473 50  0000 C CNN
+F 2 "" H 15900 4300 50  0001 C CNN
+F 3 "" H 15900 4300 50  0001 C CNN
+	1    15900 4300
+	1    0    0    -1
+$EndComp
+Wire Wire Line
+	15900 4600 15900 4350
+$Comp
+L power:PWR_FLAG #FLG?
+U 1 1 5EDD080B
+P 15900 4350
+AR Path="/5EA993EC/5EDD080B" Ref="#FLG?"  Part="1"
+AR Path="/5EAF7226/5EDD080B" Ref="#FLG?"  Part="1"
+AR Path="/5EB38D8D/5EDD080B" Ref="#FLG?"  Part="1"
+F 0 "#FLG?" H 15900 4425 50  0001 C CNN
+F 1 "PWR_FLAG" V 15900 4478 50  0000 L CNN
+F 2 "" H 15900 4350 50  0001 C CNN
+F 3 "~" H 15900 4350 50  0001 C CNN
+	1    15900 4350
+	0    1    1    0
+$EndComp
+Connection ~ 15900 4350
+Wire Wire Line
+	15900 4350 15900 4300
+$Comp
+L power:VCC #PWR?
+U 1 1 5EDD72D1
+P 11500 8200
+AR Path="/5EAF7226/5EDD72D1" Ref="#PWR?"  Part="1"
+AR Path="/5EB38D8D/5EDD72D1" Ref="#PWR?"  Part="1"
+F 0 "#PWR?" H 11500 8050 50  0001 C CNN
+F 1 "VCC" H 11517 8373 50  0000 C CNN
+F 2 "" H 11500 8200 50  0001 C CNN
+F 3 "" H 11500 8200 50  0001 C CNN
+	1    11500 8200
+	1    0    0    -1
+$EndComp
+Wire Wire Line
+	11500 8500 11500 8250
+$Comp
+L power:PWR_FLAG #FLG?
+U 1 1 5EDD72D8
+P 11500 8250
+AR Path="/5EA993EC/5EDD72D8" Ref="#FLG?"  Part="1"
+AR Path="/5EAF7226/5EDD72D8" Ref="#FLG?"  Part="1"
+AR Path="/5EB38D8D/5EDD72D8" Ref="#FLG?"  Part="1"
+F 0 "#FLG?" H 11500 8325 50  0001 C CNN
+F 1 "PWR_FLAG" V 11500 8378 50  0000 L CNN
+F 2 "" H 11500 8250 50  0001 C CNN
+F 3 "~" H 11500 8250 50  0001 C CNN
+	1    11500 8250
+	0    1    1    0
+$EndComp
+Connection ~ 11500 8250
+Wire Wire Line
+	11500 8250 11500 8200
+$Comp
+L power:GND #PWR?
+U 1 1 5EDDF24C
+P 15900 6050
+AR Path="/5EAF7226/5EDDF24C" Ref="#PWR?"  Part="1"
+AR Path="/5EB38D8D/5EDDF24C" Ref="#PWR?"  Part="1"
+F 0 "#PWR?" H 15900 5800 50  0001 C CNN
+F 1 "GND" V 15905 5922 50  0000 R CNN
+F 2 "" H 15900 6050 50  0001 C CNN
+F 3 "" H 15900 6050 50  0001 C CNN
+	1    15900 6050
+	1    0    0    -1
+$EndComp
+$Comp
+L power:PWR_FLAG #FLG?
+U 1 1 5EDDF252
+P 15900 6000
+AR Path="/5EAF7226/5EDDF252" Ref="#FLG?"  Part="1"
+AR Path="/5EB38D8D/5EDDF252" Ref="#FLG?"  Part="1"
+F 0 "#FLG?" H 15900 6075 50  0001 C CNN
+F 1 "PWR_FLAG" V 15900 6128 50  0000 L CNN
+F 2 "" H 15900 6000 50  0001 C CNN
+F 3 "~" H 15900 6000 50  0001 C CNN
+	1    15900 6000
+	0    1    1    0
+$EndComp
+Wire Wire Line
+	15900 5900 15900 6000
+Connection ~ 15900 6000
+Wire Wire Line
+	15900 6000 15900 6050
+$Comp
+L power:GND #PWR?
+U 1 1 5EDE65F4
+P 11500 9950
+AR Path="/5EAF7226/5EDE65F4" Ref="#PWR?"  Part="1"
+AR Path="/5EB38D8D/5EDE65F4" Ref="#PWR?"  Part="1"
+F 0 "#PWR?" H 11500 9700 50  0001 C CNN
+F 1 "GND" V 11505 9822 50  0000 R CNN
+F 2 "" H 11500 9950 50  0001 C CNN
+F 3 "" H 11500 9950 50  0001 C CNN
+	1    11500 9950
+	1    0    0    -1
+$EndComp
+$Comp
+L power:PWR_FLAG #FLG?
+U 1 1 5EDE65FA
+P 11500 9900
+AR Path="/5EAF7226/5EDE65FA" Ref="#FLG?"  Part="1"
+AR Path="/5EB38D8D/5EDE65FA" Ref="#FLG?"  Part="1"
+F 0 "#FLG?" H 11500 9975 50  0001 C CNN
+F 1 "PWR_FLAG" V 11500 10028 50  0000 L CNN
+F 2 "" H 11500 9900 50  0001 C CNN
+F 3 "~" H 11500 9900 50  0001 C CNN
+	1    11500 9900
+	0    1    1    0
+$EndComp
+Wire Wire Line
+	11500 9800 11500 9900
+Connection ~ 11500 9900
+Wire Wire Line
+	11500 9900 11500 9950
 $EndSCHEMATC

Commit message: Power Flags
Parts:
- gave numbers to parts that had none: 33

Commit message: Destroyed errors
Parts:
- removed U35, U38: PAL16L8, symbol Logic_Programmable:PAL16L8
- added U59, U61: PAL16L8, symbol Logic_Programmable:PAL16L8
Connections:
- net GND: now also U59.10 (GND), U61.10 (GND)
- net VCC: now also U59.20 (VCC), U61.20 (VCC)
- net at U57.1 (OEa): now also U57.19 (OEb), U59.19 (IO1)
- net at U56.1 (OE): now also U59.16 (IO4)
- net CLK: now reaches U56.11 (Cp)
- net CLK: now also U33.11 (Cp), U36.11 (Cp)
- net at U36.1 (OE): now also U59.17 (I03)
- net at U33.1 (OE): now also U59.18 (IO2)
- new net: U59.9 (I9), U61.19 (IO1)
- new net A0: U59.1 (I1)
- new net A1: U59.2 (I2)
- new net A10: U61.11 (I10)
- new net A11: U61.9 (I9)
- new net A12: U61.8 (I8)
- new net A13: U61.7 (I7)
- new net A14: U61.6 (I6)
- new net A15: U61.5 (I5)
- new net A16: U61.4 (I4)
- new net A17: U61.3 (I3)
- new net A18: U61.2 (I2)
- new net A19: U61.1 (I1)
- new net A2: U59.3 (I3)
- new net A3: U59.4 (I4)
- new net A4: U61.13 (IO7)
- new net A5: U61.14 (IO6)
- new net A6: U61.15 (IO5)
- new net A7: U61.16 (IO4)
- new net A8: U61.17 (I03)
- new net A9: U61.18 (IO2)
- no-connect marks 0 -> 10
Other:
- moved on the sheet: D1, D2, D3, D4, D5, D6, D7, D8, R10, R11, R12, R13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

Commit message: 11 errors left
Connections:
- net at U37.14 (CA): now also U34.14 (CA), U34.3 (CA), U37.3 (CA)
Changed lines of the file:
@@
 $Descr A2 23386 16535
 encoding utf-8
-Sheet 9 10
+Sheet 10 10
 Title ""
 Date ""
@@
 Wire Wire Line
 	5650 9350 6000 9350
+Wire Wire Line
+	10700 3200 10850 3200
+Wire Wire Line
+	10700 3300 10850 3300
+Wire Wire Line
+	10850 3200 10850 3300
+Wire Wire Line
+	10850 3300 10850 4500
+Connection ~ 10850 3300
+Wire Wire Line
+	10750 5900 10850 5900
+Wire Wire Line
+	10750 6000 10850 6000
+Wire Wire Line
+	10850 6000 10850 5900
+Connection ~ 10850 5900
+Wire Wire Line
+	10850 4500 11250 4500
+Connection ~ 10850 4500
+Wire Wire Line
+	10850 4500 10850 5900
 $EndSCHEMATC

Commit message: 1 Error Remains
Parts:
- added R19: 1kOhm, symbol pspice:R
Connections:
- net VCC: now also R19.1
- net at U34.14 (CA), U34.3 (CA), U37.14 (CA)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: now also R19.2
Changed lines of the file:
@@
 Wire Wire Line
 	10850 4500 10850 5900
+$Comp
+L pspice:R R19
+U 1 1 5ED917DB
+P 11500 4500
+F 0 "R19" V 11295 4500 50  0000 C CNN
+F 1 "1kOhm" V 11386 4500 50  0000 C CNN
+F 2 "" H 11500 4500 50  0001 C CNN
+F 3 "~" H 11500 4500 50  0001 C CNN
+	1    11500 4500
+	0    1    1    0
+$EndComp
+$Comp
+L power:VCC #PWR?
+U 1 1 5ED940DC
+P 11750 4500
+AR Path="/5EAF7226/5ED940DC" Ref="#PWR?"  Part="1"
+AR Path="/5EB38D8D/5ED940DC" Ref="#PWR0130"  Part="1"
+F 0 "#PWR0130" H 11750 4350 50  0001 C CNN
+F 1 "VCC" H 11767 4673 50  0000 C CNN
+F 2 "" H 11750 4500 50  0001 C CNN
+F 3 "" H 11750 4500 50  0001 C CNN
+	1    11750 4500
+	0    1    1    0
+$EndComp
 $EndSCHEMATC

Commit message: Added at least 4 Footprints
Parts:
- D1, D2, D3, D4, D5, D6, D7, D8: footprint (none) -> LED_THT:LED_D3.0mm_FlatTop
- R1, R2, R3, R4, R5, R6, R7, R8: footprint (none) -> Resistor_SMD:R_0402_1005Metric
- R10, R11, R12, R13, R14, R15, R16, R19, R9: footprint (none) -> Resistor_SMD:R_0201_0603Metric
- SW1: footprint (none) -> Button_Switch_SMD:SW_DIP_SPSTx08_Slide_Copal_CHS-08A_W5.08mm_P1.27mm_JPin
- U33, U36, U56, U57, U59, U61: footprint (none) -> Package_DIP:DIP-20_W7.62mm
Changed lines of the file:
@@
 F 0 "U57" H 19500 4081 50  0000 C CNN
 F 1 "74LS244" H 19500 3990 50  0000 C CNN
-F 2 "" H 19500 3100 50  0001 C CNN
+F 2 "Package_DIP:DIP-20_W7.62mm" H 19500 3100 50  0001 C CNN
 F 3 "http://www.ti.com/lit/gpn/sn74LS244" H 19500 3100 50  0001 C CNN
 	1    19500 3100
@@
 F 0 "SW1" H 14400 3667 50  0000 C CNN
 F 1 "SW_DIP_x08" H 14400 3576 50  0000 C CNN
-F 2 "" H 14400 3000 50  0001 C CNN
+F 2 "Button_Switch_SMD:SW_DIP_SPSTx08_Slide_Copal_CHS-08A_W5.08mm_P1.27mm_JPin" H 14400 3000 50  0001 C CNN
 F 3 "~" H 14400 3000 50  0001 C CNN
 	1    14400 3000
@@
 F 0 "R1" H 15020 2346 50  0000 L CNN
 F 1 "10kOhm" H 15020 2255 50  0000 L CNN
-F 2 "" V 14880 2300 50  0001 C CNN
+F 2 "Resistor_SMD:R_0402_1005Metric" V 14880 2300 50  0001 C CNN
 F 3 "~" H 14950 2300 50  0001 C CNN
 	1    14950 2300
@@
 F 0 "R2" H 15520 2346 50  0000 L CNN
 F 1 "10kOhm" H 15520 2255 50  0000 L CNN
-F 2 "" V 15380 2300 50  0001 C CNN
+F 2 "Resistor_SMD:R_0402_1005Metric" V 15380 2300 50  0001 C CNN
 F 3 "~" H 15450 2300 50  0001 C CNN
 	1    15450 2300
@@
 F 0 "R3" H 16020 2346 50  0000 L CNN
 F 1 "10kOhm" H 16020 2255 50  0000 L CNN
-F 2 "" V 15880 2300 50  0001 C CNN
+F 2 "Resistor_SMD:R_0402_1005Metric" V 15880 2300 50  0001 C CNN
 F 3 "~" H 15950 2300 50  0001 C CNN
 	1    15950 2300
@@
 F 0 "R4" H 16520 2346 50  0000 L CNN
 F 1 "10kOhm" H 16520 2255 50  0000 L CNN
-F 2 "" V 16380 2300 50  0001 C CNN
+F 2 "Resistor_SMD:R_0402_1005Metric" V 16380 2300 50  0001 C CNN
 F 3 "~" H 16450 2300 50  0001 C CNN
 	1    16450 2300
@@
 F 0 "R5" H 17020 2346 50  0000 L CNN
 F 1 "10kOhm" H 17020 2255 50  0000 L CNN
-F 2 "" V 16880 2300 50  0001 C CNN
+F 2 "Resistor_SMD:R_0402_1005Metric" V 16880 2300 50  0001 C CNN
 F 3 "~" H 16950 2300 50  0001 C CNN
 	1    16950 2300
@@
 F 0 "R6" H 17520 2346 50  0000 L CNN
 F 1 "10kOhm" H 17520 2255 50  0000 L CNN
-F 2 "" V 17380 2300 50  0001 C CNN
+F 2 "Resistor_SMD:R_0402_1005Metric" V 17380 2300 50  0001 C CNN
 F 3 "~" H 17450 2300 50  0001 C CNN
 	1    17450 2300
@@
 F 0 "R7" H 18020 2346 50  0000 L CNN
 F 1 "10kOhm" H 18020 2255 50  0000 L CNN
-F 2 "" V 17880 2300 50  0001 C CNN
+F 2 "Resistor_SMD:R_0402_1005Metric" V 17880 2300 50  0001 C CNN
 F 3 "~" H 17950 2300 50  0001 C CNN
 	1    17950 2300
@@
 F 0 "R8" H 18520 2346 50  0000 L CNN
 F 1 "10kOhm" H 18520 2255 50  0000 L CNN
-F 2 "" V 18380 2300 50  0001 C CNN
+F 2 "Resistor_SMD:R_0402_1005Metric" V 18380 2300 50  0001 C CNN
 F 3 "~" H 18450 2300 50  0001 C CNN
 	1    18450 2300
@@
 F 0 "U56" H 6500 9831 50  0000 C CNN
 F 1 "74LS374" H 6500 9740 50  0000 C CNN
-F 2 "" H 6500 8850 50  0001 C CNN
+F 2 "Package_DIP:DIP-20_W7.62mm" H 6500 8850 50  0001 C CNN
 F 3 "http://www.ti.com/lit/gpn/sn74LS374" H 6500 8850 50  0001 C CNN
 	1    6500 8850
@@
 F 0 "U36" H 9100 6681 50  0000 C CNN
 F 1 "74LS374" H 9100 6590 50  0000 C CNN
-F 2 "" H 9100 5700 50  0001 C CNN
+F 2 "Package_DIP:DIP-20_W7.62mm" H 9100 5700 50  0001 C CNN
 F 3 "http://www.ti.com/lit/gpn/sn74LS374" H 9100 5700 50  0001 C CNN
 	1    9100 5700
@@
 F 0 "D1" H 9243 7395 50  0000 C CNN
 F 1 "LED" H 9243 7486 50  0000 C CNN
-F 2 "" H 9250 7650 50  0001 C CNN
+F 2 "LED_THT:LED_D3.0mm_FlatTop" H 9250 7650 50  0001 C CNN
 F 3 "~" H 9250 7650 50  0001 C CNN
 	1    9250 7650
@@
 F 0 "D2" H 9243 7795 50  0000 C CNN
 F 1 "LED" H 9243 7886 50  0000 C CNN
-F 2 "" H 9250 8050 50  0001 C CNN
+F 2 "LED_THT:LED_D3.0mm_FlatTop" H 9250 8050 50  0001 C CNN
 F 3 "~" H 9250 8050 50  0001 C CNN
 	1    9250 8050
@@
 F 0 "R9" H 8620 7696 50  0000 L CNN
 F 1 "1kOhm" H 8620 7605 50  0000 L CNN
-F 2 "" V 8480 7650 50  0001 C CNN
+F 2 "Resistor_SMD:R_0201_0603Metric" V 8480 7650 50  0001 C CNN
 F 3 "~" H 8550 7650 50  0001 C CNN
 	1    8550 7650
@@
 F 0 "R10" H 8620 8096 50  0000 L CNN
 F 1 "1kOhm" H 8620 8005 50  0000 L CNN
-F 2 "" V 8480 8050 50  0001 C CNN
+F 2 "Resistor_SMD:R_0201_0603Metric" V 8480 8050 50  0001 C CNN
 F 3 "~" H 8550 8050 50  0001 C CNN
 	1    8550 8050
@@
 F 0 "D3" H 9243 8245 50  0000 C CNN
 F 1 "LED" H 9243 8336 50  0000 C CNN
-F 2 "" H 9250 8500 50  0001 C CNN
+F 2 "LED_THT:LED_D3.0mm_FlatTop" H 9250 8500 50  0001 C CNN
 F 3 "~" H 9250 8500 50  0001 C CNN
 	1    9250 8500
@@
 F 0 "D4" H 9243 8645 50  0000 C CNN
 F 1 "LED" H 9243 8736 50  0000 C CNN
-F 2 "" H 9250 8900 50  0001 C CNN
+F 2 "LED_THT:LED_D3.0mm_FlatTop" H 9250 8900 50  0001 C CNN
 F 3 "~" H 9250 8900 50  0001 C CNN
 	1    9250 8900
@@
 F 0 "R11" H 8620 8546 50  0000 L CNN
 F 1 "1kOhm" H 8620 8455 50  0000 L CNN
-F 2 "" V 8480 8500 50  0001 C CNN
+F 2 "Resistor_SMD:R_0201_0603Metric" V 8480 8500 50  0001 C CNN
 F 3 "~" H 8550 8500 50  0001 C CNN
 	1    8550 8500
@@
 F 0 "R12" H 8620 8946 50  0000 L CNN
 F 1 "1kOhm" H 8620 8855 50  0000 L CNN
-F 2 "" V 8480 8900 50  0001 C CNN
+F 2 "Resistor_SMD:R_0201_0603Metric" V 8480 8900 50  0001 C CNN
 F 3 "~" H 8550 8900 50  0001 C CNN
 	1    8550 8900
@@
 F 0 "R13" H 8670 9446 50  0000 L CNN
 F 1 "1kOhm" H 8670 9355 50  0000 L CNN
-F 2 "" V 8530 9400 50  0001 C CNN
+F 2 "Resistor_SMD:R_0201_0603Metric" V 8530 9400 50  0001 C CNN
 F 3 "~" H 8600 9400 50  0001 C CNN
 	1    8600 9400
@@
 F 0 "R14" H 8670 9846 50  0000 L CNN
 F 1 "1kOhm" H 8670 9755 50  0000 L CNN
-F 2 "" V 8530 9800 50  0001 C CNN
+F 2 "Resistor_SMD:R_0201_0603Metric" V 8530 9800 50  0001 C CNN
 F 3 "~" H 8600 9800 50  0001 C CNN
 	1    8600 9800
@@
 F 0 "R15" H 8670 10296 50  0000 L CNN
 F 1 "1kOhm" H 8670 10205 50  0000 L CNN
-F 2 "" V 8530 10250 50  0001 C CNN
+F 2 "Resistor_SMD:R_0201_0603Metric" V 8530 10250 50  0001 C CNN
 F 3 "~" H 8600 10250 50  0001 C CNN
 	1    8600 10250
@@
 F 0 "R16" H 8670 10696 50  0000 L CNN
 F 1 "1kOhm" H 8670 10605 50  0000 L CNN
-F 2 "" V 8530 10650 50  0001 C CNN
+F 2 "Resistor_SMD:R_0201_0603Metric" V 8530 10650 50  0001 C CNN
 F 3 "~" H 8600 10650 50  0001 C CNN
 	1    8600 10650
@@
 F 0 "D5" H 9293 9145 50  0000 C CNN
 F 1 "LED" H 9293 9236 50  0000 C CNN
-F 2 "" H 9300 9400 50  0001 C CNN
+F 2 "LED_THT:LED_D3.0mm_FlatTop" H 9300 9400 50  0001 C CNN
 F 3 "~" H 9300 9400 50  0001 C CNN
 	1    9300 9400
@@
 F 0 "D6" H 9293 9545 50  0000 C CNN
 F 1 "LED" H 9293 9636 50  0000 C CNN
-F 2 "" H 9300 9800 50  0001 C CNN
+F 2 "LED_THT:LED_D3.0mm_FlatTop" H 9300 9800 50  0001 C CNN
 F 3 "~" H 9300 9800 50  0001 C CNN
 	1    9300 9800
@@
 F 0 "D7" H 9293 9995 50  0000 C CNN
 F 1 "LED" H 9293 10086 50  0000 C CNN
-F 2 "" H 9300 10250 50  0001 C CNN
+F 2 "LED_THT:LED_D3.0mm_FlatTop" H 9300 10250 50  0001 C CNN
 F 3 "~" H 9300 10250 50  0001 C CNN
 	1    9300 10250
@@
 F 0 "D8" H 9293 10395 50  0000 C CNN
 F 1 "LED" H 9293 10486 50  0000 C CNN
-F 2 "" H 9300 10650 50  0001 C CNN
+F 2 "LED_THT:LED_D3.0mm_FlatTop" H 9300 10650 50  0001 C CNN
 F 3 "~" H 9300 10650 50  0001 C CNN
 	1    9300 10650
@@
 F 0 "U33" H 9050 3981 50  0000 C CNN
 F 1 "74LS374" H 9050 3890 50  0000 C CNN
-F 2 "" H 9050 3000 50  0001 C CNN
+F 2 "Package_DIP:DIP-20_W7.62mm" H 9050 3000 50  0001 C CNN
 F 3 "http://www.ti.com/lit/gpn/sn74LS374" H 9050 3000 50  0001 C CNN
 	1    9050 3000
@@
 F 0 "U61" H 6150 5331 50  0000 C CNN
 F 1 "PAL16L8" H 6150 5240 50  0000 C CNN
-F 2 "" H 6150 4450 50  0001 C CNN
+F 2 "Package_DIP:DIP-20_W7.62mm" H 6150 4450 50  0001 C CNN
 F 3 "" H 6150 4450 50  0001 C CNN
 	1    6150 4450
@@
 F 0 "U59" H 6150 3081 50  0000 C CNN
 F 1 "PAL16L8" H 6150 2990 50  0000 C CNN
-F 2 "" H 6150 2200 50  0001 C CNN
+F 2 "Package_DIP:DIP-20_W7.62mm" H 6150 2200 50  0001 C CNN
 F 3 "" H 6150 2200 50  0001 C CNN
 	1    6150 2200
@@
 F 0 "R19" V 11295 4500 50  0000 C CNN
 F 1 "1kOhm" V 11386 4500 50  0000 C CNN
-F 2 "" H 11500 4500 50  0001 C CNN
+F 2 "Resistor_SMD:R_0201_0603Metric" H 11500 4500 50  0001 C CNN
 F 3 "~" H 11500 4500 50  0001 C CNN
 	1    11500 4500

Commit message: Fixed 'Pad too close to Pad' Errors
Parts:
- R1, R2, R3, R4, R5, R6, R7, R8: footprint Resistor_SMD:R_0402_1005Metric -> Resistor_SMD:R_1206_3216Metric
- R10, R11, R12, R13, R14, R15, R16, R19, R9: footprint Resistor_SMD:R_0201_0603Metric -> Resistor_SMD:R_1206_3216Metric
Changed lines of the file:
@@
 $Descr A2 23386 16535
 encoding utf-8
-Sheet 10 10
+Sheet 9 10
 Title ""
 Date ""
@@
 F 0 "R1" H 15020 2346 50  0000 L CNN
 F 1 "10kOhm" H 15020 2255 50  0000 L CNN
-F 2 "Resistor_SMD:R_0402_1005Metric" V 14880 2300 50  0001 C CNN
+F 2 "Resistor_SMD:R_1206_3216Metric" V 14880 2300 50  0001 C CNN
 F 3 "~" H 14950 2300 50  0001 C CNN
 	1    14950 2300
@@
 F 0 "R2" H 15520 2346 50  0000 L CNN
 F 1 "10kOhm" H 15520 2255 50  0000 L CNN
-F 2 "Resistor_SMD:R_0402_1005Metric" V 15380 2300 50  0001 C CNN
+F 2 "Resistor_SMD:R_1206_3216Metric" V 15380 2300 50  0001 C CNN
 F 3 "~" H 15450 2300 50  0001 C CNN
 	1    15450 2300
@@
 F 0 "R3" H 16020 2346 50  0000 L CNN
 F 1 "10kOhm" H 16020 2255 50  0000 L CNN
-F 2 "Resistor_SMD:R_0402_1005Metric" V 15880 2300 50  0001 C CNN
+F 2 "Resistor_SMD:R_1206_3216Metric" V 15880 2300 50  0001 C CNN
 F 3 "~" H 15950 2300 50  0001 C CNN
 	1    15950 2300
@@
 F 0 "R4" H 16520 2346 50  0000 L CNN
 F 1 "10kOhm" H 16520 2255 50  0000 L CNN
-F 2 "Resistor_SMD:R_0402_1005Metric" V 16380 2300 50  0001 C CNN
+F 2 "Resistor_SMD:R_1206_3216Metric" V 16380 2300 50  0001 C CNN
 F 3 "~" H 16450 2300 50  0001 C CNN
 	1    16450 2300
@@
 F 0 "R5" H 17020 2346 50  0000 L CNN
 F 1 "10kOhm" H 17020 2255 50  0000 L CNN
-F 2 "Resistor_SMD:R_0402_1005Metric" V 16880 2300 50  0001 C CNN
+F 2 "Resistor_SMD:R_1206_3216Metric" V 16880 2300 50  0001 C CNN
 F 3 "~" H 16950 2300 50  0001 C CNN
 	1    16950 2300
@@
 F 0 "R6" H 17520 2346 50  0000 L CNN
 F 1 "10kOhm" H 17520 2255 50  0000 L CNN
-F 2 "Resistor_SMD:R_0402_1005Metric" V 17380 2300 50  0001 C CNN
+F 2 "Resistor_SMD:R_1206_3216Metric" V 17380 2300 50  0001 C CNN
 F 3 "~" H 17450 2300 50  0001 C CNN
 	1    17450 2300
@@
 F 0 "R7" H 18020 2346 50  0000 L CNN
 F 1 "10kOhm" H 18020 2255 50  0000 L CNN
-F 2 "Resistor_SMD:R_0402_1005Metric" V 17880 2300 50  0001 C CNN
+F 2 "Resistor_SMD:R_1206_3216Metric" V 17880 2300 50  0001 C CNN
 F 3 "~" H 17950 2300 50  0001 C CNN
 	1    17950 2300
@@
 F 0 "R8" H 18520 2346 50  0000 L CNN
 F 1 "10kOhm" H 18520 2255 50  0000 L CNN
-F 2 "Resistor_SMD:R_0402_1005Metric" V 18380 2300 50  0001 C CNN
+F 2 "Resistor_SMD:R_1206_3216Metric" V 18380 2300 50  0001 C CNN
 F 3 "~" H 18450 2300 50  0001 C CNN
 	1    18450 2300
@@
 F 0 "R9" H 8620 7696 50  0000 L CNN
 F 1 "1kOhm" H 8620 7605 50  0000 L CNN
-F 2 "Resistor_SMD:R_0201_0603Metric" V 8480 7650 50  0001 C CNN
+F 2 "Resistor_SMD:R_1206_3216Metric" V 8480 7650 50  0001 C CNN
 F 3 "~" H 8550 7650 50  0001 C CNN
 	1    8550 7650
@@
 F 0 "R10" H 8620 8096 50  0000 L CNN
 F 1 "1kOhm" H 8620 8005 50  0000 L CNN
-F 2 "Resistor_SMD:R_0201_0603Metric" V 8480 8050 50  0001 C CNN
+F 2 "Resistor_SMD:R_1206_3216Metric" V 8480 8050 50  0001 C CNN
 F 3 "~" H 8550 8050 50  0001 C CNN
 	1    8550 8050
@@
 F 0 "R11" H 8620 8546 50  0000 L CNN
 F 1 "1kOhm" H 8620 8455 50  0000 L CNN
-F 2 "Resistor_SMD:R_0201_0603Metric" V 8480 8500 50  0001 C CNN
+F 2 "Resistor_SMD:R_1206_3216Metric" V 8480 8500 50  0001 C CNN
 F 3 "~" H 8550 8500 50  0001 C CNN
 	1    8550 8500
@@
 F 0 "R12" H 8620 8946 50  0000 L CNN
 F 1 "1kOhm" H 8620 8855 50  0000 L CNN
-F 2 "Resistor_SMD:R_0201_0603Metric" V 8480 8900 50  0001 C CNN
+F 2 "Resistor_SMD:R_1206_3216Metric" V 8480 8900 50  0001 C CNN
 F 3 "~" H 8550 8900 50  0001 C CNN
 	1    8550 8900
@@
 F 0 "R13" H 8670 9446 50  0000 L CNN
 F 1 "1kOhm" H 8670 9355 50  0000 L CNN
-F 2 "Resistor_SMD:R_0201_0603Metric" V 8530 9400 50  0001 C CNN
+F 2 "Resistor_SMD:R_1206_3216Metric" V 8530 9400 50  0001 C CNN
 F 3 "~" H 8600 9400 50  0001 C CNN
 	1    8600 9400
@@
 F 0 "R14" H 8670 9846 50  0000 L CNN
 F 1 "1kOhm" H 8670 9755 50  0000 L CNN
-F 2 "Resistor_SMD:R_0201_0603Metric" V 8530 9800 50  0001 C CNN
+F 2 "Resistor_SMD:R_1206_3216Metric" V 8530 9800 50  0001 C CNN
 F 3 "~" H 8600 9800 50  0001 C CNN
 	1    8600 9800
@@
 F 0 "R15" H 8670 10296 50  0000 L CNN
 F 1 "1kOhm" H 8670 10205 50  0000 L CNN
-F 2 "Resistor_SMD:R_0201_0603Metric" V 8530 10250 50  0001 C CNN
+F 2 "Resistor_SMD:R_1206_3216Metric" V 8530 10250 50  0001 C CNN
 F 3 "~" H 8600 10250 50  0001 C CNN
 	1    8600 10250
@@
 F 0 "R16" H 8670 10696 50  0000 L CNN
 F 1 "1kOhm" H 8670 10605 50  0000 L CNN
-F 2 "Resistor_SMD:R_0201_0603Metric" V 8530 10650 50  0001 C CNN
+F 2 "Resistor_SMD:R_1206_3216Metric" V 8530 10650 50  0001 C CNN
 F 3 "~" H 8600 10650 50  0001 C CNN
 	1    8600 10650
@@
 F 0 "R19" V 11295 4500 50  0000 C CNN
 F 1 "1kOhm" V 11386 4500 50  0000 C CNN
-F 2 "Resistor_SMD:R_0201_0603Metric" H 11500 4500 50  0001 C CNN
+F 2 "Resistor_SMD:R_1206_3216Metric" H 11500 4500 50  0001 C CNN
 F 3 "~" H 11500 4500 50  0001 C CNN
 	1    11500 4500
