File: Proj_5/LED_Switch.sch (KiCad schematic (older format))
At the start: 34 parts, among them SW1 SW_DIP_x08, U33 74LS374, U34 MAN72A, U36 74LS374, U37 MAN72A, U56 74LS374, U57 74LS244, U59 PAL16L8, U61 PAL16L8

Commit message: Cool pt2
Changed lines of the file:
@@
 	1    0    0    -1
 $EndComp
-Wire Wire Line
-	14100 2600 14100 2700
-Connection ~ 14100 2700
-Wire Wire Line
-	14100 2700 14100 2800
-Connection ~ 14100 2800
-Wire Wire Line
-	14100 2800 14100 2900
-Connection ~ 14100 2900
-Wire Wire Line
-	14100 2900 14100 3000
-Connection ~ 14100 3000
-Wire Wire Line
-	14100 3000 14100 3100
-Connection ~ 14100 3100
-Wire Wire Line
-	14100 3100 14100 3200
-Connection ~ 14100 3200
-Wire Wire Line
-	14100 3200 14100 3300
-Connection ~ 14100 3300
 $Comp
 L power:VCC #PWR?
@@
 L power:GND #PWR?
 U 1 1 5EB7EBB7
-P 14100 3650
+P 14100 2600
 AR Path="/5EAF7226/5EB7EBB7" Ref="#PWR?"  Part="1"
 AR Path="/5EB38D8D/5EB7EBB7" Ref="#PWR038"  Part="1"
-F 0 "#PWR038" H 14100 3400 50  0001 C CNN
-F 1 "GND" V 14105 3522 50  0000 R CNN
-F 2 "" H 14100 3650 50  0001 C CNN
-F 3 "" H 14100 3650 50  0001 C CNN
-	1    14100 3650
-	1    0    0    -1
+F 0 "#PWR038" H 14100 2350 50  0001 C CNN
+F 1 "GND" V 14105 2472 50  0000 R CNN
+F 2 "" H 14100 2600 50  0001 C CNN
+F 3 "" H 14100 2600 50  0001 C CNN
+	1    14100 2600
+	0    1    1    0
 $EndComp
 Wire Wire Line
@@
 Wire Wire Line
 	9100 6500 9100 6650
-Wire Wire Line
-	14100 3300 14100 3650
 Wire Wire Line
 	9800 7500 9950 7500
@@
 	0    1    1    0
 $EndComp
+$Comp
+L power:GND #PWR?
+U 1 1 5EBF1165
+P 14100 3300
+AR Path="/5EAF7226/5EBF1165" Ref="#PWR?"  Part="1"
+AR Path="/5EB38D8D/5EBF1165" Ref="#PWR?"  Part="1"
+F 0 "#PWR?" H 14100 3050 50  0001 C CNN
+F 1 "GND" V 14105 3172 50  0000 R CNN
+F 2 "" H 14100 3300 50  0001 C CNN
+F 3 "" H 14100 3300 50  0001 C CNN
+	1    14100 3300
+	0    1    1    0
+$EndComp
+$Comp
+L power:GND #PWR?
+U 1 1 5EBF167B
+P 14100 3200
+AR Path="/5EAF7226/5EBF167B" Ref="#PWR?"  Part="1"
+AR Path="/5EB38D8D/5EBF167B" Ref="#PWR?"  Part="1"
+F 0 "#PWR?" H 14100 2950 50  0001 C CNN
+F 1 "GND" V 14105 3072 50  0000 R CNN
+F 2 "" H 14100 3200 50  0001 C CNN
+F 3 "" H 14100 3200 50  0001 C CNN
+	1    14100 3200
+	0    1    1    0
+$EndComp
+$Comp
+L power:GND #PWR?
+U 1 1 5EBF1A5E
+P 14100 3100
+AR Path="/5EAF7226/5EBF1A5E" Ref="#PWR?"  Part="1"
+AR Path="/5EB38D8D/5EBF1A5E" Ref="#PWR?"  Part="1"
+F 0 "#PWR?" H 14100 2850 50  0001 C CNN
+F 1 "GND" V 14105 2972 50  0000 R CNN
+F 2 "" H 14100 3100 50  0001 C CNN
+F 3 "" H 14100 3100 50  0001 C CNN
+	1    14100 3100
+	0    1    1    0
+$EndComp
+$Comp
+L power:GND #PWR?
+U 1 1 5EBF1F00
+P 14100 3000
+AR Path="/5EAF7226/5EBF1F00" Ref="#PWR?"  Part="1"
+AR Path="/5EB38D8D/5EBF1F00" Ref="#PWR?"  Part="1"
+F 0 "#PWR?" H 14100 2750 50  0001 C CNN
+F 1 "GND" V 14105 2872 50  0000 R CNN
+F 2 "" H 14100 3000 50  0001 C CNN
+F 3 "" H 14100 3000 50  0001 C CNN
+	1    14100 3000
+	0    1    1    0
+$EndComp
+$Comp
+L power:GND #PWR?
+U 1 1 5EBF2497
+P 14100 2900
+AR Path="/5EAF7226/5EBF2497" Ref="#PWR?"  Part="1"
+AR Path="/5EB38D8D/5EBF2497" Ref="#PWR?"  Part="1"
+F 0 "#PWR?" H 14100 2650 50  0001 C CNN
+F 1 "GND" V 14105 2772 50  0000 R CNN
+F 2 "" H 14100 2900 50  0001 C CNN
+F 3 "" H 14100 2900 50  0001 C CNN
+	1    14100 2900
+	0    1    1    0
+$EndComp
+$Comp
+L power:GND #PWR?
+U 1 1 5EBF2A88
+P 14100 2800
+AR Path="/5EAF7226/5EBF2A88" Ref="#PWR?"  Part="1"
+AR Path="/5EB38D8D/5EBF2A88" Ref="#PWR?"  Part="1"
+F 0 "#PWR?" H 14100 2550 50  0001 C CNN
+F 1 "GND" V 14105 2672 50  0000 R CNN
+F 2 "" H 14100 2800 50  0001 C CNN
+F 3 "" H 14100 2800 50  0001 C CNN
+	1    14100 2800
+	0    1    1    0
+$EndComp
+$Comp
+L power:GND #PWR?
+U 1 1 5EBF2FD7
+P 14100 2700
+AR Path="/5EAF7226/5EBF2FD7" Ref="#PWR?"  Part="1"
+AR Path="/5EB38D8D/5EBF2FD7" Ref="#PWR?"  Part="1"
+F 0 "#PWR?" H 14100 2450 50  0001 C CNN
+F 1 "GND" V 14105 2572 50  0000 R CNN
+F 2 "" H 14100 2700 50  0001 C CNN
+F 3 "" H 14100 2700 50  0001 C CNN
+	1    14100 2700
+	0    1    1    0
+$EndComp
