File: Proj_5/Proj_5.kicad_pcb (KiCad board)
At the start: 4 copper layers, 717.5 x 762 mm, 132 parts, among them J1 Conn_02x15_Top_Bottom, J10 Conn_02x20_Counter_Clockwise, J2 Conn_02x15_Top_Bottom, J3 Conn_02x15_Top_Bottom, J4 Conn_02x07_Counter_Clockwise, J5 Conn_02x04_Top_Bottom, J6 Conn_02x06_Counter_Clockwise, J7 DSUB-9, J8 Conn_01x02, J9 Conn_02x16_Counter_Clockwise, SW1 SW_DIP_x08, SW10 Switch_SW_SPST, SW11 Switch_SW_SPST, SW12 Switch_SW_SPST, SW13 Switch_SW_SPST, SW14 Switch_SW_SPST, SW15 Switch_SW_SPST, SW16 Switch_SW_SPST, SW17 Switch_SW_SPST, SW18 Switch_SW_SPST, SW19 Switch_SW_SPST, SW2 Shift, SW20 Switch_SW_SPST, SW21 Switch_SW_SPST, SW22 Switch_SW_SPST, SW23 Switch_SW_SPST, SW24 NMI Button, SW25 Reset Button, SW26 IR0 Button, SW3 Switch_SW_SPST, SW4 Switch_SW_SPST, SW5 Switch_SW_SPST, SW6 Switch_SW_SPST, SW7 CTRL, SW8 Switch_SW_SPST, SW9 Switch_SW_SPST, U1 8255, U10 8259, U11 8254, U12 28F010, U13 PAL16L8, U14 16550, U15 PAL16L8, U16 PAL16L8, U17 pkd8279, U18 74LS138, U19 8086_Min_Mode, U2 8255, U20 74LS373, U21 74LS373, U22 74LS244, U23 74LS373, U24 74LS245, U25 74LS245, U3 8255, U33 74LS374, U34 MAN72A, U35 PAL16L8, U36 74LS374, U37 MAN72A, U38 PAL16L8, U39 PAL16L8, U4 28F010, U40 PAL16L8, U48 MAX6816, U49 MAX6816, U5 CY7C199, U50 MAX6816, U51 PAL16L8, U52 PAL16L8, U55 max235cpg, U56 74LS374, U57 74LS244, U59 PAL16L8, U6 CY7C199, U61 PAL16L8, U7 PAL16L8, U8 CY7C199, U9 CY7C199

Commit message: Data Aquired
Parts:
- moved U22 563.0 mm to (586.1, 212.1)
- moved C22 485.7 mm to (618.6, 386.7)
- moved DS1 485.7 mm to (621.7, 377.2)
- moved C1 324.5 mm to (529.7, 295.3)
- moved C3 324.5 mm to (529.7, 299.7)
- moved C4 324.5 mm to (529.6, 290.8)
- moved C5 324.5 mm to (529.5, 304.2)
- moved C6 324.5 mm to (529.6, 308.6)
- moved U24 321.3 mm to (224.8, 134.6), turned to 270 degrees
- moved U20 280.2 mm to (487.7, -27.9)
- moved U25 256.7 mm to (189.2, 105.4), turned to 270 degrees
- moved C11 244.8 mm to (501.6, 10.1)
- moved C13 244.8 mm to (519.2, -8.24)
- moved U21 196.8 mm to (125.7, 97.8), turned to 180 degrees
- moved C21 195.2 mm to (542.4, 89.1)
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Connections:
- U8 pad 11: /D0 -> /D8
- U8 pad 12: /D1 -> /D9
- U8 pad 13: /D2 -> /D10
- U8 pad 15: /D3 -> /D11
- U8 pad 16: /D4 -> /D12
- U8 pad 17: /D5 -> /D13
- U8 pad 18: /D6 -> /D14
- U8 pad 19: /D7 -> /D15
- U9 pad 11: /D0 -> /D8
- U9 pad 12: /D1 -> /D9
- U9 pad 13: /D2 -> /D10
- U9 pad 15: /D3 -> /D11
- U9 pad 16: /D4 -> /D12
- U9 pad 17: /D5 -> /D13
- U9 pad 18: /D6 -> /D14
- U9 pad 19: /D7 -> /D15
Routing:
- net /D0: track 205.2 -> 662.4 mm, vias 2 -> 6
- net /D2: track 193.6 -> 650.0 mm, vias 2 -> 10
- net /D1: track 197.8 -> 654.3 mm, vias 2 -> 10
- net /D8: track 187.7 -> 569.4 mm, vias 2 -> 6
- net /D9: track 183.4 -> 564.1 mm, vias 2 -> 10
- net /D10: track 180.0 -> 559.4 mm, vias 2 -> 10
- net /D11: track 153.7 -> 494.4 mm, vias 1 -> 5
- net /D12: track 154.3 -> 491.9 mm, vias 1 -> 7
- net /D13: track 154.9 -> 489.3 mm, vias 1 -> 7
- net /D14: track 156.8 -> 488.1 mm, vias 1 -> 7
- net /D15: track 158.7 -> 486.5 mm, vias 1 -> 5
- net /D7: track 301.6 -> 594.6 mm, vias 5 -> 9
- net /D6: track 302.0 -> 592.2 mm, vias 5 -> 9
- net /D5: track 303.2 -> 591.5 mm, vias 4 -> 8
- net /D4: track 316.1 -> 602.5 mm, vias 4 -> 8
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
Commit message: Fixed 'Pad too close to Pad' Errors
Parts:
- CLK_R1, CLK_R2, R10, R11, R12, R13, R14, R15, R16, R17, R19, R9: footprint Resistor_SMD:R_0201_0603Metric -> Resistor_SMD:R_0805_2012Metric
- J1, J2, J3: footprint Connector_PinHeader_1.00mm:PinHeader_2x15_P1.00mm_Vertical -> Connector_PinHeader_2.54mm:PinHeader_2x15_P2.54mm_Vertical
- J10: footprint Connector_PinHeader_1.00mm:PinHeader_2x20_P1.00mm_Vertical -> Connector_PinHeader_2.54mm:PinHeader_2x20_P2.54mm_Vertical
- J4: footprint Connector_PinHeader_1.00mm:PinHeader_2x07_P1.00mm_Vertical -> Connector_PinHeader_2.54mm:PinHeader_2x07_P2.54mm_Vertical
- J5: footprint Connector_PinHeader_1.00mm:PinHeader_2x04_P1.00mm_Vertical -> Connector_PinHeader_2.54mm:PinHeader_2x04_P2.54mm_Vertical
- J6: footprint Connector_PinHeader_1.00mm:PinHeader_2x06_P1.00mm_Vertical -> Connector_PinHeader_2.54mm:PinHeader_2x06_P2.54mm_Vertical
- J8: footprint Connector_PinHeader_1.00mm:PinHeader_1x02_P1.00mm_Vertical -> Connector_PinHeader_2.54mm:PinHeader_1x02_P2.54mm_Vertical
- J9: footprint Connector_PinHeader_1.00mm:PinHeader_2x16_P1.00mm_Vertical -> Connector_PinHeader_2.54mm:PinHeader_2x16_P2.54mm_Vertical
- R1, R2, R3, R4, R5, R6, R7, R8: footprint Resistor_SMD:R_0402_1005Metric -> Resistor_SMD:R_0805_2012Metric
- moved J5 24.3 mm to (85.1, 325.1), turned to 180 degrees
- moved J4 21.6 mm to (24.1, 444.5)
- moved J10 14.1 mm to (442.0, -71.1)
- moved J8 12.0 mm to (556.3, 96.5)
- moved J9 4.56 mm to (532.1, 86.4)
Routing:
- net Net-(J5-Pad1): track 25.9 -> 6.04 mm
- net Net-(J5-Pad3): track 22.9 -> 4.62 mm
- net Net-(J5-Pad5): track 20.0 -> 3.21 mm
- net Net-(J5-Pad7): track 17.7 -> 1.33 mm
- net Net-(J5-Pad6): track 0.60 -> 0.00 mm

Commit message: Finished Address Bus + Address and Data Bus Enables
Parts:
- moved U13 510.8 mm to (236.2, -168.9)
- moved U15 510.8 mm to (172.7, -168.9)
- moved U16 510.8 mm to (234.9, -203.2)
- moved U38 510.8 mm to (276.3, -186.1)
- moved U39 510.8 mm to (210.8, -203.2)
- moved U40 510.8 mm to (207.0, -168.9)
- moved U51 510.8 mm to (181.6, -203.2)
- moved U52 510.8 mm to (157.5, -203.2)
- moved U35 510.8 mm to (265.4, -186.1)
- moved U20 365.5 mm to (125.7, -78.7)
- moved U23 58.9 mm to (133.3, -12.7)
- moved J6 41.8 mm to (477.5, 120.7)
- moved J2 16.3 mm to (640.1, 63.5)
Routing:
- net Net-(J6-Pad2): track 0.00 -> 291.0 mm, vias 0 -> 2
- net Net-(J6-Pad1): track 0.00 -> 286.6 mm, vias 0 -> 2
- net Net-(J6-Pad3): track 0.00 -> 254.5 mm, vias 0 -> 4
- net /A15: track 211.5 -> 420.3 mm
- net /A14: track 583.8 -> 790.8 mm
- net /A13: track 564.2 -> 769.3 mm
- net /A12: track 449.4 -> 652.8 mm
- net /A11: track 498.2 -> 699.8 mm
- net /A10: track 480.1 -> 679.9 mm
- net /A9: track 472.1 -> 670.1 mm
- net /A8: track 479.9 -> 676.1 mm
- net /A7: track 376.2 -> 494.3 mm
- net /~BHE: track 103.4 -> 221.0 mm, vias 1 -> 3
- net /A6: track 414.0 -> 530.3 mm
- net /A16: track 184.4 -> 299.3 mm, vias 2 -> 4
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
Commit message: More Headers - 690 to 540 No-Connects
Parts:
- moved J9 545.6 mm to (-5.08, 181.6)
- moved J10 444.2 mm to (1.27, -127.0)
- moved J7 144.8 mm to (535.9, -247.7)
- moved J5 89.6 mm to (1.27, 356.9)
- moved R19 35.9 mm to (425.4, 372.1)
- moved J8 30.7 mm to (532.1, 77.5)
- moved U11 24.5 mm to (57.1, 444.5)
- moved U33 24.0 mm to (419.1, 405.1), turned to 270 degrees
- moved J4 16.5 mm to (24.1, 461.0)
- moved U34 15.1 mm to (405.1, 379.7)
- moved U36 13.7 mm to (448.3, 405.1), turned to 270 degrees
- moved J1 13.3 mm to (631.2, -61.0)
- moved R8 11.7 mm to (295.9, 448.3)
- moved C21 11.5 mm to (547.4, 78.7), turned to 270 degrees
- moved J2 8.98 mm to (631.2, 62.2)
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Connections:
- U11 pad 10: Net-(J4-Pad3) -> Net-(J4-Pad2)
- U11 pad 11: Net-(J4-Pad2) -> Net-(J4-Pad3)
Routing:
- net /D0: track 662.4 -> 929.9 mm, vias 6 -> 9
- net /D3: track 610.3 -> 871.2 mm
- net /D4: track 602.5 -> 859.5 mm
- net /D2: track 650.0 -> 906.9 mm
- net /D1: track 654.3 -> 908.9 mm, vias 10 -> 11
- net /D7: track 594.6 -> 830.9 mm, vias 9 -> 11
- net /D6: track 592.2 -> 825.9 mm, vias 9 -> 11
- net /D5: track 591.5 -> 818.6 mm
- net /D8: track 569.4 -> 720.7 mm
- net /D14: track 488.1 -> 639.3 mm
- net /D10: track 559.4 -> 710.6 mm
- net /D12: track 491.9 -> 643.2 mm
- net /D13: track 489.3 -> 639.4 mm
- net /D9: track 564.1 -> 712.4 mm
- net /D11: track 494.4 -> 642.7 mm
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
Commit message: Fixed 8255 Headers + Control Bus Header
Parts:
- moved J6 511.1 mm to (1.27, -64.8)
- moved U22 487.7 mm to (191.8, -74.9), turned to 90 degrees
- moved C14 407.7 mm to (160.0, -52.1)
- moved J8 224.5 mm to (692.1, 234.9)
- moved C21 208.0 mm to (683.3, 236.2)
- moved C2 117.0 mm to (405.7, 45.1)
- moved C7 117.0 mm to (384.0, 65.3)
- moved C8 117.0 mm to (375.8, 65.3)
- moved C9 117.0 mm to (379.9, 65.3)
- moved CLK_Gen1 117.0 mm to (395.0, 45.1)
- moved CLK_R1 117.0 mm to (415.3, 54.0)
- moved CLK_R2 117.0 mm to (416.6, 42.5)
- moved OSC1 117.0 mm to (415.3, 48.9)
Routing:
- net /~WR: track 335.7 -> 634.8 mm, vias 4 -> 6
- net Net-(J6-Pad1): track 286.6 -> 563.2 mm, vias 2 -> 7
- net Net-(J6-Pad2): track 291.0 -> 565.9 mm, vias 2 -> 7
- net /~RD: track 338.5 -> 613.0 mm, vias 9 -> 11
- net /8279, 8259, 8254/~INTA: track 27.9 -> 268.6 mm, vias 0 -> 4
- net Net-(J6-Pad11): track 0.00 -> 226.2 mm, vias 0 -> 4
- net /8279, 8259, 8254/INT: track 47.4 -> 266.3 mm, vias 0 -> 2
- net /M~IO: track 0.00 -> 218.5 mm, vias 0 -> 2
- net /D0: track 929.9 -> 1101.7 mm
- net /D1: track 908.9 -> 1069.2 mm
- net /D2: track 906.9 -> 1055.8 mm
- net Net-(J6-Pad3): track 254.5 -> 392.7 mm, vias 4 -> 6
- net /D3: track 871.2 -> 1008.6 mm
- net /D4: track 859.5 -> 985.5 mm
- net /D5: track 818.6 -> 933.1 mm
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
Commit message: UART Connections + Some other Stuff
Parts:
- moved C2 11.8 mm to (398.8, 35.6)
- moved OSC1 7.67 mm to (422.9, 49.8)
- moved CLK_R1 2.99 mm to (417.8, 55.5), turned to 90 degrees
- turned CLK_R2 to 270 degrees
Routing:
- net /8279, 8259, 8254/~INTA: track 268.6 -> 798.8 mm, vias 4 -> 9
- net /~RD: track 613.0 -> 1131.0 mm, vias 11 -> 16
- net /~WR: track 634.8 -> 1149.3 mm, vias 6 -> 11
- net /M~IO: track 218.5 -> 660.6 mm, vias 2 -> 5
- net Net-(J7-Pad6): track 0.00 -> 119.9 mm, vias 0 -> 2
- net Net-(J7-Pad1): track 0.00 -> 117.9 mm, vias 0 -> 2
- net Net-(J7-Pad7): track 0.00 -> 112.4 mm, vias 0 -> 2
- net Net-(J7-Pad4): track 0.00 -> 101.5 mm, vias 0 -> 2
- net Net-(J7-Pad8): track 0.00 -> 100.9 mm, vias 0 -> 2
- net Net-(U14-Pad10): track 0.00 -> 66.9 mm
- net Net-(J7-Pad3): track 0.00 -> 60.5 mm
- net Net-(U14-Pad11): track 0.00 -> 48.5 mm
- net Net-(J7-Pad2): track 0.00 -> 48.4 mm
- net Net-(CLK_Gen1-Pad17): track 0.00 -> 27.5 mm, vias 0 -> 2
- net Net-(CLK_Gen1-Pad16): track 0.00 -> 26.4 mm
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
Commit message: Pals Hooked up to Address Bus
Parts:
- moved U7 387.6 mm to (224.8, -210.8), turned to 270 degrees
- moved R2 383.3 mm to (45.7, 133.3)
- moved R8 383.3 mm to (77.5, 133.3)
- moved R1 383.3 mm to (40.6, 133.3)
- moved R3 383.3 mm to (50.8, 133.3)
- moved R4 383.3 mm to (55.9, 133.3)
- moved R5 383.3 mm to (61.0, 133.3)
- moved R6 383.3 mm to (66.0, 133.3)
- moved R7 383.3 mm to (72.4, 133.3)
- moved SW1 383.3 mm to (30.5, 151.8)
- moved U57 383.3 mm to (91.4, 141.0)
- moved U52 365.8 mm to (520.7, -246.4)
- moved U51 339.1 mm to (520.7, -208.3)
- moved U39 233.8 mm to (444.5, -210.8), turned to 270 degrees
- moved U61 227.1 mm to (273.1, -210.8), turned to 270 degrees
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Routing:
- net /A19: track 196.2 -> 1046.5 mm, vias 4 -> 10
- net /A18: track 200.0 -> 1039.1 mm, vias 4 -> 10
- net /A17: track 193.3 -> 1021.7 mm, vias 4 -> 10
- net /A9: track 766.9 -> 1564.0 mm, vias 12 -> 16
- net /A8: track 777.3 -> 1560.3 mm, vias 12 -> 16
- net /A16: track 390.2 -> 1170.7 mm, vias 6 -> 11
- net /A15: track 509.5 -> 1280.8 mm, vias 4 -> 9
- net /A10: track 778.5 -> 1511.7 mm, vias 10 -> 14
- net /A14: track 884.2 -> 1607.7 mm, vias 5 -> 9
- net /A13: track 861.1 -> 1575.3 mm, vias 13 -> 17
- net /A7: track 593.6 -> 1303.8 mm, vias 10 -> 14
- net /A12: track 748.8 -> 1453.9 mm, vias 13 -> 17
- net /A6: track 633.9 -> 1337.4 mm, vias 11 -> 15
- net /A11: track 794.1 -> 1494.1 mm, vias 11 -> 15
- net /A5: track 611.5 -> 1308.2 mm, vias 13 -> 17
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
Commit message: Cool pt2
Parts:
- moved C1 426.7 mm to (107.4, 356.2)
- moved C3 426.7 mm to (107.4, 360.7)
- moved C4 426.7 mm to (107.3, 351.8)
- moved C5 426.7 mm to (107.2, 365.1)
- moved C6 426.7 mm to (107.3, 369.6)
- moved U36 396.6 mm to (76.2, 268.0), turned to 90 degrees
- moved C22 390.8 mm to (228.0, 401.3)
- moved DS1 390.8 mm to (231.1, 391.8)
- moved U37 354.8 mm to (90.2, 293.4), turned to 180 degrees
- moved U33 342.4 mm to (105.4, 268.0), turned to 90 degrees
- moved R19 332.7 mm to (101.6, 295.9), turned to 90 degrees
- moved U34 298.5 mm to (119.4, 293.4), turned to 180 degrees
- moved D1 228.0 mm to (8.89, 210.2)
- moved D2 228.0 mm to (8.89, 217.8)
- moved D3 228.0 mm to (8.89, 225.4)
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Routing:
- net /M~IO: track 660.6 -> 1298.2 mm, vias 5 -> 8
- net /D2: track 1060.4 -> 1565.5 mm, vias 10 -> 27
- net /D1: track 1074.0 -> 1576.4 mm, vias 11 -> 28
- net /D7: track 927.1 -> 1427.9 mm, vias 11 -> 26
- net /D0: track 1107.0 -> 1606.9 mm, vias 9 -> 18
- net /D6: track 933.1 -> 1426.6 mm, vias 11 -> 30
- net /D5: track 937.0 -> 1422.3 mm, vias 8 -> 27
- net /D4: track 989.6 -> 1466.7 mm, vias 8 -> 27
- net /D3: track 1012.9 -> 1482.5 mm, vias 6 -> 23
- net /~WR: track 1093.4 -> 1420.1 mm, vias 11 -> 13
- net /~RD: track 1075.1 -> 1393.9 mm, vias 16 -> 18
- net Net-(U10-Pad18): track 0.00 -> 161.0 mm
- net /8279, 8259, 8254/RESET: track 0.00 -> 159.2 mm
- net GND: track 101.4 -> 39.9 mm, vias 6 -> 5
- net Net-(J5-Pad7): track 68.9 -> 14.9 mm
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- added copper zone on GND, net GND
- added copper zone on VCC, net VCC
