File: Proj_5/Proj_5.kicad_pcb (KiCad board)
At the start: 4 copper layers, 717.5 x 762 mm, 132 parts, among them J1 Conn_02x15_Top_Bottom, J10 Conn_02x20_Counter_Clockwise, J2 Conn_02x15_Top_Bottom, J3 Conn_02x15_Top_Bottom, J4 Conn_02x07_Counter_Clockwise, J5 Conn_02x04_Top_Bottom, J6 Conn_02x06_Counter_Clockwise, J7 DSUB-9, J8 Conn_01x02, J9 Conn_02x16_Counter_Clockwise, SW1 SW_DIP_x08, SW10 Switch_SW_SPST, SW11 Switch_SW_SPST, SW12 Switch_SW_SPST, SW13 Switch_SW_SPST, SW14 Switch_SW_SPST, SW15 Switch_SW_SPST, SW16 Switch_SW_SPST, SW17 Switch_SW_SPST, SW18 Switch_SW_SPST, SW19 Switch_SW_SPST, SW2 Shift, SW20 Switch_SW_SPST, SW21 Switch_SW_SPST, SW22 Switch_SW_SPST, SW23 Switch_SW_SPST, SW24 NMI Button, SW25 Reset Button, SW26 IR0 Button, SW3 Switch_SW_SPST, SW4 Switch_SW_SPST, SW5 Switch_SW_SPST, SW6 Switch_SW_SPST, SW7 CTRL, SW8 Switch_SW_SPST, SW9 Switch_SW_SPST, U1 8255, U10 8259, U11 8254, U12 28F010, U13 PAL16L8, U14 16550, U15 PAL16L8, U16 PAL16L8, U17 pkd8279, U18 74LS138, U19 8086_Min_Mode, U2 8255, U20 74LS373, U21 74LS373, U22 74LS244, U23 74LS373, U24 74LS245, U25 74LS245, U3 8255, U33 74LS374, U34 MAN72A, U35 PAL16L8, U36 74LS374, U37 MAN72A, U38 PAL16L8, U39 PAL16L8, U4 28F010, U40 PAL16L8, U48 MAX6816, U49 MAX6816, U5 CY7C199, U50 MAX6816, U51 PAL16L8, U52 PAL16L8, U55 max235cpg, U56 74LS374, U57 74LS244, U59 PAL16L8, U6 CY7C199, U61 PAL16L8, U7 PAL16L8, U8 CY7C199, U9 CY7C199

Commit message: addresses baby
Parts:
- moved C13 464.1 mm to (144.1, 314.3), turned to 270 degrees
- moved C10 263.7 mm to (617.2, -158.1), turned to 90 degrees
- moved R17 21.0 mm to (252.7, 320.7), turned to 90 degrees
- moved C2 1.27 mm to (262.9, -45.7), turned to 180 degrees
Routing:
- net /~BHE: track 889.3 -> 1441.5 mm, vias 6 -> 10
- net /A14: track 1607.7 -> 2155.4 mm, vias 9 -> 16
- net /A13: track 1575.3 -> 2121.2 mm, vias 17 -> 24
- net /A12: track 1453.9 -> 1997.8 mm, vias 17 -> 24
- net /A11: track 1494.1 -> 2036.2 mm, vias 15 -> 22
- net /A10: track 1511.7 -> 2051.8 mm, vias 14 -> 21
- net /A9: track 1564.0 -> 2102.3 mm, vias 16 -> 23
- net /A8: track 1560.3 -> 2095.9 mm, vias 16 -> 21
- net /A7: track 1303.8 -> 1809.9 mm, vias 14 -> 19
- net /A6: track 1337.4 -> 1841.3 mm, vias 15 -> 20
- net /A5: track 1308.2 -> 1810.5 mm, vias 17 -> 22
- net /A4: track 1300.5 -> 1781.4 mm, vias 17 -> 22
- net /A3: track 1233.7 -> 1711.8 mm, vias 15 -> 20
- net /A2: track 1223.2 -> 1698.5 mm, vias 14 -> 19
- net /A15: track 1280.8 -> 1744.1 mm, vias 9 -> 16
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