File: Part1_Schematic/Proj_5/16550UART.sch (KiCad schematic (older format))
At the start: 10 parts, among them J7 DSUB-9, U14 16550, U51 PAL16L8, U52 74AHC1G02, U53 74LVC1G08, U54 74AHC1G02, U55 max235cpg

Commit message: Addressing for 8279 and 8259
Parts:
- renumbered C20 to C?, J7 to J?, R18 to R?, U55 to U?, U51 to U?, U52 to U?, U54 to U?, U53 to U?
Connections:
- net GND: now also U?.21 (SHDN); no longer U?.10 (GND), U?.20 (*EN)
- net VCC: now also U?.20 (*EN); no longer C?.1, U?.12 (VCC), U?.20 (VCC)
- net D10 renamed D2
- net D11 renamed D3
- net D12 renamed D4
- net D13 renamed D5
- net D14 renamed D6
- net D15 renamed D7
- net D8 renamed D0
- net D9 renamed D1
- new net +5V: C?.1, U?.12 (VCC)
- no-connect marks 32 -> 31
Other:
- note added: "235 Needs Enables But from where"
Changed lines of the file:
@@
 $Descr A2 23386 16535
 encoding utf-8
-Sheet 8 10
+Sheet 9 9
 Title ""
 Date ""
@@
 P 19000 7100
 AR Path="/5EAF7226/5EA3C31E" Ref="J?"  Part="1"
-AR Path="/5EA98A67/5EA3C31E" Ref="J7"  Part="1"
-F 0 "J7" H 19828 6753 60  0000 L CNN
+AR Path="/5EA98A67/5EA3C31E" Ref="J?"  Part="1"
+F 0 "J?" H 19828 6753 60  0000 L CNN
 F 1 "DSUB-9" H 19828 6647 60  0000 L CNN
 F 2 "DSUB-9" H 19600 6740 60  0001 C CNN
@@
 P 14050 7000
 AR Path="/5EAF7226/5EA3C324" Ref="U?"  Part="1"
-AR Path="/5EA98A67/5EA3C324" Ref="U55"  Part="1"
-F 0 "U55" H 15350 7387 60  0000 C CNN
+AR Path="/5EA98A67/5EA3C324" Ref="U?"  Part="1"
+F 0 "U?" H 15350 7387 60  0000 C CNN
 F 1 "max235cpg" H 15350 7281 60  0000 C CNN
 F 2 "max235cpg" H 15350 7240 60  0001 C CNN
@@
 P 15000 8600
 AR Path="/5EAF7226/5EA40B25" Ref="#PWR?"  Part="1"
-AR Path="/5EA98A67/5EA40B25" Ref="#PWR098"  Part="1"
-F 0 "#PWR098" H 15000 8350 50  0001 C CNN
+AR Path="/5EA98A67/5EA40B25" Ref="#PWR?"  Part="1"
+F 0 "#PWR?" H 15000 8350 50  0001 C CNN
 F 1 "GND" H 15005 8427 50  0000 C CNN
 F 2 "" H 15000 8600 50  0001 C CNN
@@
 P 9200 9300
 AR Path="/5EAF7226/5EA41175" Ref="#PWR?"  Part="1"
-AR Path="/5EA98A67/5EA41175" Ref="#PWR095"  Part="1"
-F 0 "#PWR095" H 9200 9050 50  0001 C CNN
+AR Path="/5EA98A67/5EA41175" Ref="#PWR?"  Part="1"
+F 0 "#PWR?" H 9200 9050 50  0001 C CNN
 F 1 "GND" H 9205 9127 50  0000 C CNN
 F 2 "" H 9200 9300 50  0001 C CNN
@@
 P 10650 5650
 AR Path="/5EAF7226/5EA41CE6" Ref="#PWR?"  Part="1"
-AR Path="/5EA98A67/5EA41CE6" Ref="#PWR096"  Part="1"
-F 0 "#PWR096" H 10650 5400 50  0001 C CNN
+AR Path="/5EA98A67/5EA41CE6" Ref="#PWR?"  Part="1"
+F 0 "#PWR?" H 10650 5400 50  0001 C CNN
 F 1 "GND" H 10655 5477 50  0000 C CNN
 F 2 "" H 10650 5650 50  0001 C CNN
@@
 NoConn ~ 8200 8500
 NoConn ~ 8200 8600
+$Comp
+L power:+5V #PWR?
+U 1 1 5EA81CD6
+P 15700 9250
+F 0 "#PWR?" H 15700 9100 50  0001 C CNN
+F 1 "+5V" V 15715 9378 50  0000 L CNN
+F 2 "" H 15700 9250 50  0001 C CNN
+F 3 "" H 15700 9250 50  0001 C CNN
+	1    15700 9250
+	-1   0    0    1
+$EndComp
 Wire Wire Line
 	15700 8600 15600 8600
 Connection ~ 15700 8600
+Wire Wire Line
+	15700 8600 15700 9250
 $Comp
 L power:GND #PWR?
@@
 P 16100 8600
 AR Path="/5EAF7226/5EA3C332" Ref="#PWR?"  Part="1"
-AR Path="/5EA98A67/5EA3C332" Ref="#PWR0100"  Part="1"
-F 0 "#PWR0100" H 16100 8350 50  0001 C CNN
+AR Path="/5EA98A67/5EA3C332" Ref="#PWR?"  Part="1"
+F 0 "#PWR?" H 16100 8350 50  0001 C CNN
 F 1 "GND" H 16105 8427 50  0000 C CNN
 F 2 "" H 16100 8600 50  0001 C CNN
@@
 AR Path="/5EA98353/5EA3C32A" Ref="C?"  Part="1"
 AR Path="/5EAF7226/5EA3C32A" Ref="C?"  Part="1"
-AR Path="/5EA98A67/5EA3C32A" Ref="C20"  Part="1"
-F 0 "C20" V 15698 8600 50  0000 C CNN
+AR Path="/5EA98A67/5EA3C32A" Ref="C?"  Part="1"
+F 0 "C?" V 15698 8600 50  0000 C CNN
 F 1 "0.1uF" V 15789 8600 50  0000 C CNN
 F 2 "" H 15988 8450 50  0001 C CNN
@@
 P 19550 8200
 AR Path="/5EAF7226/5EAA0E88" Ref="#PWR?"  Part="1"
-AR Path="/5EA98A67/5EAA0E88" Ref="#PWR0106"  Part="1"
-F 0 "#PWR0106" H 19550 7950 50  0001 C CNN
+AR Path="/5EA98A67/5EAA0E88" Ref="#PWR?"  Part="1"
+F 0 "#PWR?" H 19550 7950 50  0001 C CNN
 F 1 "GND" H 19555 8027 50  0000 C CNN
 F 2 "" H 19550 8200 50  0001 C CNN
@@
 Text HLabel 8200 8700 0    50   Input ~ 0
 ~RD
+Text HLabel 8200 6900 0    50   BiDi ~ 0
+D7
+Text HLabel 8200 6800 0    50   BiDi ~ 0
+D6
+Text HLabel 8200 6700 0    50   BiDi ~ 0
+D5
+Text HLabel 8200 6600 0    50   BiDi ~ 0
+D4
+Text HLabel 8200 6500 0    50   BiDi ~ 0
+D3
+Text HLabel 8200 6400 0    50   BiDi ~ 0
+D2
+Text HLabel 8200 6300 0    50   BiDi ~ 0
+D1
+Text HLabel 8200 6200 0    50   BiDi ~ 0
+D0
 Wire Wire Line
 	8200 8800 7850 8800
@@
 P 7850 8800
 AR Path="/5EAF7226/5EAA4D1F" Ref="#PWR?"  Part="1"
-AR Path="/5EA98A67/5EAA4D1F" Ref="#PWR093"  Part="1"
-F 0 "#PWR093" H 7850 8550 50  0001 C CNN
+AR Path="/5EA98A67/5EAA4D1F" Ref="#PWR?"  Part="1"
+F 0 "#PWR?" H 7850 8550 50  0001 C CNN
 F 1 "GND" H 7855 8627 50  0000 C CNN
 F 2 "" H 7850 8800 50  0001 C CNN
@@
 NoConn ~ 10200 7300
 NoConn ~ 10200 7000
+Text Notes 13100 10400 0    118  ~ 0
+235 Needs Enables But from where
 NoConn ~ 8200 7800
 NoConn ~ 8200 8100
@@
 A2
 $Comp
-L Logic_Programmable:PAL16L8 U51
+L Logic_Programmable:PAL16L8 U?
 U 1 1 5EA83B43
 P 5400 7250
-F 0 "U51" H 5400 8131 50  0000 C CNN
+F 0 "U?" H 5400 8131 50  0000 C CNN
 F 1 "PAL16L8" H 5400 8040 50  0000 C CNN
 F 2 "" H 5400 7250 50  0001 C CNN
@@
 A0
 $Comp
-L 74xGxx:74AHC1G02 U52
+L 74xGxx:74AHC1G02 U?
 U 1 1 5EA8FF70
 P 6250 5750
-F 0 "U52" V 6179 5880 50  0000 L CNN
+F 0 "U?" V 6179 5880 50  0000 L CNN
 F 1 "74AHC1G02" V 6270 5880 50  0000 L CNN
 F 2 "" H 6250 5750 50  0001 C CNN
@@
 $EndComp
 $Comp
-L 74xGxx:74AHC1G02 U54
+L 74xGxx:74AHC1G02 U?
 U 1 1 5EA96A09
 P 6950 5750
-F 0 "U54" V 6879 5880 50  0000 L CNN
+F 0 "U?" V 6879 5880 50  0000 L CNN
 F 1 "74AHC1G02" V 6970 5880 50  0000 L CNN
 F 2 "" H 6950 5750 50  0001 C CNN
@@
 $EndComp
 $Comp
-L 74xGxx:74LVC1G08 U53
+L 74xGxx:74LVC1G08 U?
 U 1 1 5EA99D66
 P 6600 6300
-F 0 "U53" V 6529 6430 50  0000 L CNN
+F 0 "U?" V 6529 6430 50  0000 L CNN
 F 1 "74LVC1G08" V 6620 6430 50  0000 L CNN
 F 2 "" H 6600 6300 50  0001 C CNN
@@
 	5900 7600 5900 7450
 $Comp
-L power:VCC #PWR092
+L power:VCC #PWR?
 U 1 1 5EAA2831
 P 7400 7400
-F 0 "#PWR092" H 7400 7250 50  0001 C CNN
+F 0 "#PWR?" H 7400 7250 50  0001 C CNN
 F 1 "VCC" H 7417 7573 50  0000 C CNN
 F 2 "" H 7400 7400 50  0001 C CNN
@@
 	7950 7500 7950 7400
 $Comp
-L Device:R R18
+L Device:R R?
 U 1 1 5EAA6766
 P 7550 7400
-F 0 "R18" V 7343 7400 50  0000 C CNN
+F 0 "R?" V 7343 7400 50  0000 C CNN
 F 1 "1K" V 7434 7400 50  0000 C CNN
 F 2 "" V 7480 7400 50  0001 C CNN
@@
 NoConn ~ 5900 6850
 NoConn ~ 5900 6950
+$Comp
+L power:GND #PWR?
+U 1 1 5EAB604F
+P 16650 7000
+F 0 "#PWR?" H 16650 6750 50  0001 C CNN
+F 1 "GND" V 16655 6872 50  0000 R CNN
+F 2 "" H 16650 7000 50  0001 C CNN
+F 3 "" H 16650 7000 50  0001 C CNN
+	1    16650 7000
+	0    -1   -1   0
+$EndComp
+$Comp
+L power:VCC #PWR?
+U 1 1 5EAB6B80
+P 14050 7000
+F 0 "#PWR?" H 14050 6850 50  0001 C CNN
+F 1 "VCC" H 14067 7173 50  0000 C CNN
+F 2 "" H 14050 7000 50  0001 C CNN
+F 3 "" H 14050 7000 50  0001 C CNN
+	1    14050 7000
+	1    0    0    -1
+$EndComp
 Wire Wire Line
 	9200 5200 9200 5650
 $Comp
-L power:VCC #PWR094
+L power:VCC #PWR?
 U 1 1 5F0AFF2A
 P 9200 5200
-F 0 "#PWR094" H 9200 5050 50  0001 C CNN
+F 0 "#PWR?" H 9200 5050 50  0001 C CNN
 F 1 "VCC" H 9217 5373 50  0000 C CNN
 F 2 "" H 9200 5200 50  0001 C CNN
@@
 	1    0    0    -1
 $EndComp
-Text HLabel 8200 6200 0    50   BiDi ~ 0
-D8
-Text HLabel 8200 6300 0    50   BiDi ~ 0
-D9
-Text HLabel 8200 6400 0    50   BiDi ~ 0
-D10
-Text HLabel 8200 6500 0    50   BiDi ~ 0
-D11
-Text HLabel 8200 6600 0    50   BiDi ~ 0
-D12
-Text HLabel 8200 6700 0    50   BiDi ~ 0
-D13
-Text HLabel 8200 6800 0    50   BiDi ~ 0
-D14
-Text HLabel 8200 6900 0    50   BiDi ~ 0
-D15
-Wire Wire Line
-	5400 6550 5200 6550
-Wire Wire Line
-	5200 6550 5200 6300
-Wire Wire Line
-	5400 7850 5400 8000
-$Comp
-L power:VCC #PWR029
-U 1 1 5EDADCA7
-P 5200 6300
-F 0 "#PWR029" H 5200 6150 50  0001 C CNN
-F 1 "VCC" H 5217 6473 50  0000 C CNN
-F 2 "" H 5200 6300 50  0001 C CNN
-F 3 "" H 5200 6300 50  0001 C CNN
-	1    5200 6300
-	1    0    0    -1
-$EndComp
-$Comp
-L power:GND #PWR?
-U 1 1 5EDB05EC
-P 5400 8000
-AR Path="/5EAF7226/5EDB05EC" Ref="#PWR?"  Part="1"
-AR Path="/5EA98A67/5EDB05EC" Ref="#PWR030"  Part="1"
-F 0 "#PWR030" H 5400 7750 50  0001 C CNN
-F 1 "GND" H 5405 7827 50  0000 C CNN
-F 2 "" H 5400 8000 50  0001 C CNN
-F 3 "" H 5400 8000 50  0001 C CNN
-	1    5400 8000
-	1    0    0    -1
-$EndComp
-$Comp
-L power:VCC #PWR031
-U 1 1 5EDC0795
-P 15700 9600
-F 0 "#PWR031" H 15700 9450 50  0001 C CNN
-F 1 "VCC" H 15717 9773 50  0000 C CNN
-F 2 "" H 15700 9600 50  0001 C CNN
-F 3 "" H 15700 9600 50  0001 C CNN
-	1    15700 9600
-	-1   0    0    1
-$EndComp
-Wire Wire Line
-	15700 8600 15700 9600
-$Comp
-L power:GND #PWR?
-U 1 1 5F37E591
-P 14050 7000
-F 0 "#PWR?" H 14050 6750 50  0001 C CNN
-F 1 "GND" V 14055 6872 50  0000 R CNN
-F 2 "" H 14050 7000 50  0001 C CNN
-F 3 "" H 14050 7000 50  0001 C CNN
-	1    14050 7000
-	0    1    1    0
-$EndComp
-NoConn ~ 16650 7000
 $EndSCHEMATC
