File: Part1_Schematic/Proj_5/8086_Demuxing.sch (KiCad schematic (older format))
At the start: 11 parts, among them J6 Conn_02x30_Top_Bottom, J8 Conn_01x02, U19 8086_Min_Mode, U20 74LS373, U21 74LS373, U22 74LS244, U23 74LS373, U24 74LS245, U25 74LS245

Commit message: Addressing for 8279 and 8259
Parts:
- removed C21: 100uF, symbol Device:C
- removed J8: Conn_01x02, symbol Connector_Generic:Conn_01x02
- renumbered J6 to J?
Connections:
- wire segments 410 -> 411
- no-connect marks 21 -> 6
Changed lines of the file:
@@
 $Descr A2 23386 16535
 encoding utf-8
-Sheet 7 10
+Sheet 8 9
 Title ""
 Date ""
@@
 	11050 8100 11050 7950
 Wire Wire Line
+	11050 7950 11150 7950
+Wire Wire Line
 	13400 8100 13600 8100
 Wire Wire Line
@@
 L power:GND #PWR0126
 U 1 1 5EC40EB5
-P 11500 7950
-F 0 "#PWR0126" H 11500 7700 50  0001 C CNN
-F 1 "GND" H 11505 7777 50  0000 C CNN
-F 2 "" H 11500 7950 50  0001 C CNN
-F 3 "" H 11500 7950 50  0001 C CNN
-	1    11500 7950
+P 11150 7950
+F 0 "#PWR0126" H 11150 7700 50  0001 C CNN
+F 1 "GND" H 11155 7777 50  0000 C CNN
+F 2 "" H 11150 7950 50  0001 C CNN
+F 3 "" H 11150 7950 50  0001 C CNN
+	1    11150 7950
 	0    -1   -1   0
 $EndComp
@@
 L power:GND #PWR0127
 U 1 1 5ECB05B8
-P 10450 11850
-F 0 "#PWR0127" H 10450 11600 50  0001 C CNN
-F 1 "GND" H 10455 11677 50  0000 C CNN
-F 2 "" H 10450 11850 50  0001 C CNN
-F 3 "" H 10450 11850 50  0001 C CNN
-	1    10450 11850
+P 10750 11850
+F 0 "#PWR0127" H 10750 11600 50  0001 C CNN
+F 1 "GND" H 10755 11677 50  0000 C CNN
+F 2 "" H 10750 11850 50  0001 C CNN
+F 3 "" H 10750 11850 50  0001 C CNN
+	1    10750 11850
 	0    1    1    0
 $EndComp
@@
 Wire Wire Line
 	7850 6550 7850 6900
+Wire Wire Line
+	7850 6100 7850 6150
 Connection ~ 7850 6550
 $Comp
@@
 NMI_IN
 $Comp
-L Connector_Generic:Conn_02x30_Top_Bottom J6
+L Connector_Generic:Conn_02x30_Top_Bottom J?
 U 1 1 5EDA27EF
 P 13050 3050
-F 0 "J6" H 13100 4667 50  0000 C CNN
+F 0 "J?" H 13100 4667 50  0000 C CNN
 F 1 "Conn_02x30_Top_Bottom" H 13100 4576 50  0000 C CNN
 F 2 "" H 13050 3050 50  0001 C CNN
@@
 	3500 3500 3500 13250
 Wire Wire Line
+	7150 9100 3600 9100
+Wire Wire Line
+	3600 9100 3600 3550
+Wire Wire Line
+	3600 3550 12050 3550
+Wire Wire Line
+	12050 3550 12050 3350
+Wire Wire Line
+	7150 8900 3700 8900
+Wire Wire Line
+	3700 8900 3700 3600
+Wire Wire Line
+	3700 3600 11950 3600
+Wire Wire Line
+	11950 3600 11950 3350
+Wire Wire Line
+	7150 8400 3800 8400
+Wire Wire Line
+	3800 8400 3800 3650
+Wire Wire Line
+	3800 3650 11850 3650
+Wire Wire Line
+	11850 3650 11850 3350
+Wire Wire Line
 	7150 8100 3900 8100
 Wire Wire Line
 	3900 8100 3900 3700
 Wire Wire Line
+	3900 3700 11750 3700
+Wire Wire Line
+	11750 3700 11750 3350
+Wire Wire Line
 	7150 7400 4000 7400
 Wire Wire Line
 	4000 7400 4000 3750
+Wire Wire Line
+	4000 3750 11650 3750
+Wire Wire Line
+	11650 3750 11650 3350
 Wire Wire Line
 	20450 8900 20450 500
@@
 	13250 2500 13350 2500
 $Comp
-L power:GND #PWR089
+L power:GND #PWR?
 U 1 1 5F5023A7
 P 14450 2500
-F 0 "#PWR089" H 14450 2250 50  0001 C CNN
+F 0 "#PWR?" H 14450 2250 50  0001 C CNN
 F 1 "GND" H 14455 2327 50  0000 C CNN
 F 2 "" H 14450 2500 50  0001 C CNN
@@
 Connection ~ 14450 2500
 $Comp
-L power:VCC #PWR084
+L power:VCC #PWR?
 U 1 1 5EF73B7F
 P 7850 6100
-F 0 "#PWR084" H 7850 5950 50  0001 C CNN
+F 0 "#PWR?" H 7850 5950 50  0001 C CNN
 F 1 "VCC" H 7867 6273 50  0000 C CNN
 F 2 "" H 7850 6100 50  0001 C CNN
@@
 	1    0    0    -1
 $EndComp
-$Comp
-L power:VCC #PWR085
+Wire Wire Line
+	9500 7150 9500 7600
+$Comp
+L power:VCC #PWR?
 U 1 1 5EF74C0E
-P 9600 6950
-F 0 "#PWR085" H 9600 6800 50  0001 C CNN
-F 1 "VCC" H 9617 7123 50  0000 C CNN
-F 2 "" H 9600 6950 50  0001 C CNN
-F 3 "" H 9600 6950 50  0001 C CNN
-	1    9600 6950
-	0    1    1    0
+P 9500 7150
+F 0 "#PWR?" H 9500 7000 50  0001 C CNN
+F 1 "VCC" H 9517 7323 50  0000 C CNN
+F 2 "" H 9500 7150 50  0001 C CNN
+F 3 "" H 9500 7150 50  0001 C CNN
+	1    9500 7150
+	1    0    0    -1
 $EndComp
 Wire Wire Line
 	12100 7150 12100 7600
 $Comp
-L power:VCC #PWR088
+L power:VCC #PWR?
 U 1 1 5EF9EA73
 P 12100 7150
-F 0 "#PWR088" H 12100 7000 50  0001 C CNN
+F 0 "#PWR?" H 12100 7000 50  0001 C CNN
 F 1 "VCC" H 12117 7323 50  0000 C CNN
 F 2 "" H 12100 7150 50  0001 C CNN
@@
 	16900 7600 17350 7600
 $Comp
-L power:VCC #PWR091
+L power:VCC #PWR?
 U 1 1 5EFC96F5
 P 16900 7600
-F 0 "#PWR091" H 16900 7450 50  0001 C CNN
+F 0 "#PWR?" H 16900 7450 50  0001 C CNN
 F 1 "VCC" H 16917 7773 50  0000 C CNN
 F 2 "" H 16900 7600 50  0001 C CNN
@@
 	0    -1   -1   0
 $EndComp
-$Comp
-L power:VCC #PWR090
+Wire Wire Line
+	16400 9400 15950 9400
+$Comp
+L power:VCC #PWR?
 U 1 1 5EFF3F9C
-P 16600 9500
-F 0 "#PWR090" H 16600 9350 50  0001 C CNN
-F 1 "VCC" H 16617 9673 50  0000 C CNN
-F 2 "" H 16600 9500 50  0001 C CNN
-F 3 "" H 16600 9500 50  0001 C CNN
-	1    16600 9500
-	-1   0    0    1
+P 16400 9400
+F 0 "#PWR?" H 16400 9250 50  0001 C CNN
+F 1 "VCC" H 16417 9573 50  0000 C CNN
+F 2 "" H 16400 9400 50  0001 C CNN
+F 3 "" H 16400 9400 50  0001 C CNN
+	1    16400 9400
+	0    1    1    0
 $EndComp
 Wire Wire Line
 	10850 10650 11300 10650
 $Comp
-L power:VCC #PWR087
+L power:VCC #PWR?
 U 1 1 5F01F222
 P 10850 10650
-F 0 "#PWR087" H 10850 10500 50  0001 C CNN
+F 0 "#PWR?" H 10850 10500 50  0001 C CNN
 F 1 "VCC" H 10867 10823 50  0000 C CNN
 F 2 "" H 10850 10650 50  0001 C CNN
@@
 	9750 3950 10200 3950
 $Comp
-L power:VCC #PWR086
+L power:VCC #PWR?
 U 1 1 5F04A79B
 P 9750 3950
-F 0 "#PWR086" H 9750 3800 50  0001 C CNN
+F 0 "#PWR?" H 9750 3800 50  0001 C CNN
 F 1 "VCC" H 9767 4123 50  0000 C CNN
 F 2 "" H 9750 3950 50  0001 C CNN
 F 3 "" H 9750 3950 50  0001 C CNN
 	1    9750 3950
-	-1   0    0    1
-$EndComp
+	0    -1   -1   0
+$EndComp
+$Comp
+L power:PWR_FLAG #FLG?
+U 1 1 5F179D43
+P 7850 6150
+AR Path="/5EA045EA/5F179D43" Ref="#FLG?"  Part="1"
+AR Path="/5EA98353/5EA34234/5F179D43" Ref="#FLG?"  Part="1"
+AR Path="/5E9F3A3D/5F179D43" Ref="#FLG?"  Part="1"
+F 0 "#FLG?" H 7850 6225 50  0001 C CNN
+F 1 "PWR_FLAG" V 7850 6277 50  0000 L CNN
+F 2 "" H 7850 6150 50  0001 C CNN
+F 3 "~" H 7850 6150 50  0001 C CNN
+	1    7850 6150
+	0    1    1    0
+$EndComp
+Connection ~ 7850 6150
+Wire Wire Line
+	7850 6150 7850 6550
 Wire Wire Line
 	8550 10250 10100 10250
@@
 	4200 13150 4200 3800
 Wire Wire Line
-	12050 3700 12050 3350
-Wire Wire Line
-	3900 3700 12050 3700
-Wire Wire Line
-	11950 3750 11950 3350
-Wire Wire Line
-	4000 3750 11950 3750
-Wire Wire Line
-	11850 3800 11850 3350
-Wire Wire Line
-	4200 3800 11850 3800
-NoConn ~ 7150 8400
-NoConn ~ 7150 8900
-NoConn ~ 7150 9100
-Wire Wire Line
-	11050 7950 11500 7950
-Wire Wire Line
-	10750 11850 10450 11850
-NoConn ~ 10750 11350
-NoConn ~ 10750 11450
-NoConn ~ 10750 11550
-NoConn ~ 10750 11650
-NoConn ~ 11750 11350
-NoConn ~ 11750 11450
-NoConn ~ 11750 11550
-NoConn ~ 11750 11650
-NoConn ~ 10750 11950
-Wire Wire Line
-	16600 9400 16600 9500
-Wire Wire Line
-	15950 9400 16600 9400
-Wire Wire Line
-	9500 6950 9600 6950
-Wire Wire Line
-	9500 6950 9500 7600
-NoConn ~ 11750 3350
-NoConn ~ 11650 3350
-NoConn ~ 11550 3350
-$Comp
-L Connector_Generic:Conn_01x02 J8
-U 1 1 5EEC8283
-P 3250 1500
-F 0 "J8" H 3168 1175 50  0000 C CNN
-F 1 "Conn_01x02" H 3168 1266 50  0000 C CNN
-F 2 "" H 3250 1500 50  0001 C CNN
-F 3 "~" H 3250 1500 50  0001 C CNN
-	1    3250 1500
-	-1   0    0    1
-$EndComp
-$Comp
-L power:VCC #PWR022
-U 1 1 5EEC8F27
-P 4000 1200
-F 0 "#PWR022" H 4000 1050 50  0001 C CNN
-F 1 "VCC" H 4017 1373 50  0000 C CNN
-F 2 "" H 4000 1200 50  0001 C CNN
-F 3 "" H 4000 1200 50  0001 C CNN
-	1    4000 1200
-	1    0    0    -1
-$EndComp
-$Comp
-L Device:C C?
-U 1 1 5EFA8610
-P 4500 1500
-AR Path="/5EA98353/5EFA8610" Ref="C?"  Part="1"
-AR Path="/5E9F3A3D/5EFA8610" Ref="C21"  Part="1"
-F 0 "C21" V 4248 1500 50  0000 C CNN
-F 1 "100uF" V 4339 1500 50  0000 C CNN
-F 2 "" H 4538 1350 50  0001 C CNN
-F 3 "~" H 4500 1500 50  0001 C CNN
-	1    4500 1500
-	-1   0    0    1
-$EndComp
-$Comp
-L power:GND #PWR023
-U 1 1 5EFA8616
-P 4500 1700
-F 0 "#PWR023" H 4500 1450 50  0001 C CNN
-F 1 "GND" H 4505 1527 50  0000 C CNN
-F 2 "" H 4500 1700 50  0001 C CNN
-F 3 "" H 4500 1700 50  0001 C CNN
-	1    4500 1700
-	1    0    0    -1
-$EndComp
-Wire Wire Line
-	4500 1350 4300 1350
-Wire Wire Line
-	4300 1350 4300 1400
-Wire Wire Line
-	3450 1400 4000 1400
-Connection ~ 4000 1400
-Wire Wire Line
-	4000 1400 4300 1400
-Wire Wire Line
-	4150 1500 4150 1650
-Wire Wire Line
-	4150 1650 4500 1650
-Wire Wire Line
-	3450 1500 4150 1500
-Wire Wire Line
-	4500 1650 4500 1700
-Connection ~ 4500 1650
-Wire Wire Line
-	7850 6100 7850 6550
-Wire Wire Line
-	4000 1200 4000 1400
+	4200 3800 11550 3800
+Wire Wire Line
+	11550 3800 11550 3350
 $EndSCHEMATC
