File: Part1_Schematic/Proj_5/8279_59_54.sch (KiCad schematic (older format))
At the start: 44 parts, among them J4 Conn_02x07_Counter_Clockwise, J5 Conn_02x07_Counter_Clockwise, SW10 Switch_SW_SPST, SW11 Switch_SW_SPST, SW12 Switch_SW_SPST, SW13 Switch_SW_SPST, SW14 Switch_SW_SPST, SW15 Switch_SW_SPST, SW16 Switch_SW_SPST, SW17 Switch_SW_SPST, SW18 Switch_SW_SPST, SW19 Switch_SW_SPST, SW2 Shift, SW20 Switch_SW_SPST, SW21 Switch_SW_SPST, SW22 Switch_SW_SPST, SW23 Switch_SW_SPST, SW24 NMI Button, SW25 Reset Button, SW26 IR0 Button, SW3 Switch_SW_SPST, SW4 Switch_SW_SPST, SW5 Switch_SW_SPST, SW6 Switch_SW_SPST, SW7 CTRL, SW8 Switch_SW_SPST, SW9 Switch_SW_SPST, U10 8259, U11 8254, U17 pkd8279, U18 74LS138, U48 MAX6816, U49 MAX6816, U50 MAX6816

Commit message: Addressing for 8279 and 8259
Parts:
- removed U?: PAL16L8, symbol Logic_Programmable:PAL16L8
- removed U?: 74LVC1G11, symbol 74xGxx:74LVC1G11
- removed U?: 74LVC1G08, symbol 74xGxx:74LVC1G08
- renumbered C19 to C?, C18 to C?, C15 to C?, C11 to C?, J5 to J?, J4 to J?, R17 to R?, SW24 to SW?, SW25 to SW?, SW26 to SW?, U48 to U?, U49 to U?, U50 to U?
Connections:
- net GND: now also C?.2; no longer U17.20 (VSS)
- net at U17.22 (~CS): no longer U10.1 (~CS~)
- net A1: no longer names the net of U17.21 (A0)
- net A1: no longer U10.27 (A0)
- no-connect marks 22 -> 16
Other:
- note added: "Needs VCC Pins, Headers, Decoding"
- note removed: "Needs: Decoding"
