File: Part1_Schematic/Proj_5/CY7C199.sch (KiCad schematic (older format))
At the start: 10 parts, among them U5 CY7C199, U6 CY7C199, U7 PAL16L8, U8 CY7C199, U9 CY7C199

Commit message: Addressing for 8279 and 8259
Parts:
- renumbered C4 to C?, C1 to C?, C3 to C?, C5 to C?, C6 to C?
Connections:
- net GND: no longer U7.10 (GND)
Changed lines of the file:
@@
 $Descr A2 23386 16535
 encoding utf-8
-Sheet 3 10
+Sheet 3 9
 Title ""
 Date ""
@@
 P 4950 9000
 AR Path="/5E9F3A3D/5F07F2BC" Ref="#PWR?"  Part="1"
-AR Path="/5EA98353/5F07F2BC" Ref="#PWR07"  Part="1"
-F 0 "#PWR07" H 4950 8850 50  0001 C CNN
+AR Path="/5EA98353/5F07F2BC" Ref="#PWR?"  Part="1"
+F 0 "#PWR?" H 4950 8850 50  0001 C CNN
 F 1 "VCC" H 4967 9173 50  0000 C CNN
 F 2 "" H 4950 9000 50  0001 C CNN
@@
 P 10000 9000
 AR Path="/5E9F3A3D/5F08872C" Ref="#PWR?"  Part="1"
-AR Path="/5EA98353/5F08872C" Ref="#PWR017"  Part="1"
-F 0 "#PWR017" H 10000 8850 50  0001 C CNN
+AR Path="/5EA98353/5F08872C" Ref="#PWR?"  Part="1"
+F 0 "#PWR?" H 10000 8850 50  0001 C CNN
 F 1 "VCC" H 10017 9173 50  0000 C CNN
 F 2 "" H 10000 9000 50  0001 C CNN
@@
 P 10000 5400
 AR Path="/5E9F3A3D/5F091CCD" Ref="#PWR?"  Part="1"
-AR Path="/5EA98353/5F091CCD" Ref="#PWR016"  Part="1"
-F 0 "#PWR016" H 10000 5250 50  0001 C CNN
+AR Path="/5EA98353/5F091CCD" Ref="#PWR?"  Part="1"
+F 0 "#PWR?" H 10000 5250 50  0001 C CNN
 F 1 "VCC" H 10017 5573 50  0000 C CNN
 F 2 "" H 10000 5400 50  0001 C CNN
@@
 P 4950 5400
 AR Path="/5E9F3A3D/5F09B239" Ref="#PWR?"  Part="1"
-AR Path="/5EA98353/5F09B239" Ref="#PWR04"  Part="1"
-F 0 "#PWR04" H 4950 5250 50  0001 C CNN
+AR Path="/5EA98353/5F09B239" Ref="#PWR?"  Part="1"
+F 0 "#PWR?" H 4950 5250 50  0001 C CNN
 F 1 "VCC" H 4967 5573 50  0000 C CNN
 F 2 "" H 4950 5400 50  0001 C CNN
@@
 P 7150 3250
 AR Path="/5E9F3A3D/5F0A4C11" Ref="#PWR?"  Part="1"
-AR Path="/5EA98353/5F0A4C11" Ref="#PWR014"  Part="1"
-F 0 "#PWR014" H 7150 3100 50  0001 C CNN
+AR Path="/5EA98353/5F0A4C11" Ref="#PWR?"  Part="1"
+F 0 "#PWR?" H 7150 3100 50  0001 C CNN
 F 1 "VCC" H 7167 3423 50  0000 C CNN
 F 2 "" H 7150 3250 50  0001 C CNN
@@
 $EndComp
 $Comp
-L Device:C C4
+L Device:C C?
 U 1 1 5F0B1B35
 P 7750 3600
-AR Path="/5EA98353/5F0B1B35" Ref="C4"  Part="1"
+AR Path="/5EA98353/5F0B1B35" Ref="C?"  Part="1"
 AR Path="/5EA98A67/5F0B1B35" Ref="C?"  Part="1"
-F 0 "C4" V 7498 3600 50  0000 C CNN
+F 0 "C?" V 7498 3600 50  0000 C CNN
 F 1 "0.1uF" V 7589 3600 50  0000 C CNN
 F 2 "" H 7788 3450 50  0001 C CNN
@@
 AR Path="/5EAF7226/5F0B1B3B" Ref="#PWR?"  Part="1"
 AR Path="/5EA98A67/5F0B1B3B" Ref="#PWR?"  Part="1"
-AR Path="/5EA98353/5F0B1B3B" Ref="#PWR015"  Part="1"
-F 0 "#PWR015" H 7900 3350 50  0001 C CNN
+AR Path="/5EA98353/5F0B1B3B" Ref="#PWR?"  Part="1"
+F 0 "#PWR?" H 7900 3350 50  0001 C CNN
 F 1 "GND" H 7905 3427 50  0000 C CNN
 F 2 "" H 7900 3600 50  0001 C CNN
@@
 	7150 3600 6450 3600
 $Comp
-L Device:C C1
+L Device:C C?
 U 1 1 5F0DC280
 P 5100 5150
-AR Path="/5EA98353/5F0DC280" Ref="C1"  Part="1"
+AR Path="/5EA98353/5F0DC280" Ref="C?"  Part="1"
 AR Path="/5EA98A67/5F0DC280" Ref="C?"  Part="1"
-F 0 "C1" V 4848 5150 50  0000 C CNN
+F 0 "C?" V 4848 5150 50  0000 C CNN
 F 1 "0.1uF" V 4939 5150 50  0000 C CNN
 F 2 "" H 5138 5000 50  0001 C CNN
@@
 AR Path="/5EAF7226/5F0DC286" Ref="#PWR?"  Part="1"
 AR Path="/5EA98A67/5F0DC286" Ref="#PWR?"  Part="1"
-AR Path="/5EA98353/5F0DC286" Ref="#PWR08"  Part="1"
-F 0 "#PWR08" H 5100 4750 50  0001 C CNN
+AR Path="/5EA98353/5F0DC286" Ref="#PWR?"  Part="1"
+F 0 "#PWR?" H 5100 4750 50  0001 C CNN
 F 1 "GND" H 5105 4827 50  0000 C CNN
 F 2 "" H 5100 5000 50  0001 C CNN
@@
 	5100 5400 5400 5400
 $Comp
-L Device:C C3
+L Device:C C?
 U 1 1 5F10F8DC
 P 5150 8750
-AR Path="/5EA98353/5F10F8DC" Ref="C3"  Part="1"
+AR Path="/5EA98353/5F10F8DC" Ref="C?"  Part="1"
 AR Path="/5EA98A67/5F10F8DC" Ref="C?"  Part="1"
-F 0 "C3" V 4898 8750 50  0000 C CNN
+F 0 "C?" V 4898 8750 50  0000 C CNN
 F 1 "0.1uF" V 4989 8750 50  0000 C CNN
 F 2 "" H 5188 8600 50  0001 C CNN
@@
 AR Path="/5EAF7226/5F10F8E2" Ref="#PWR?"  Part="1"
 AR Path="/5EA98A67/5F10F8E2" Ref="#PWR?"  Part="1"
-AR Path="/5EA98353/5F10F8E2" Ref="#PWR013"  Part="1"
-F 0 "#PWR013" H 5150 8350 50  0001 C CNN
+AR Path="/5EA98353/5F10F8E2" Ref="#PWR?"  Part="1"
+F 0 "#PWR?" H 5150 8350 50  0001 C CNN
 F 1 "GND" H 5155 8427 50  0000 C CNN
 F 2 "" H 5150 8600 50  0001 C CNN
@@
 	5150 9000 5400 9000
 $Comp
-L Device:C C5
+L Device:C C?
 U 1 1 5F11B32F
 P 10200 5150
-AR Path="/5EA98353/5F11B32F" Ref="C5"  Part="1"
+AR Path="/5EA98353/5F11B32F" Ref="C?"  Part="1"
 AR Path="/5EA98A67/5F11B32F" Ref="C?"  Part="1"
-F 0 "C5" V 9948 5150 50  0000 C CNN
+F 0 "C?" V 9948 5150 50  0000 C CNN
 F 1 "0.1uF" V 10039 5150 50  0000 C CNN
 F 2 "" H 10238 5000 50  0001 C CNN
@@
 AR Path="/5EAF7226/5F11B335" Ref="#PWR?"  Part="1"
 AR Path="/5EA98A67/5F11B335" Ref="#PWR?"  Part="1"
-AR Path="/5EA98353/5F11B335" Ref="#PWR018"  Part="1"
-F 0 "#PWR018" H 10200 4750 50  0001 C CNN
+AR Path="/5EA98353/5F11B335" Ref="#PWR?"  Part="1"
+F 0 "#PWR?" H 10200 4750 50  0001 C CNN
 F 1 "GND" H 10205 4827 50  0000 C CNN
 F 2 "" H 10200 5000 50  0001 C CNN
@@
 	10200 5300 10200 5400
 $Comp
-L Device:C C6
+L Device:C C?
 U 1 1 5F125E11
 P 10250 8750
-AR Path="/5EA98353/5F125E11" Ref="C6"  Part="1"
+AR Path="/5EA98353/5F125E11" Ref="C?"  Part="1"
 AR Path="/5EA98A67/5F125E11" Ref="C?"  Part="1"
-F 0 "C6" V 9998 8750 50  0000 C CNN
+F 0 "C?" V 9998 8750 50  0000 C CNN
 F 1 "0.1uF" V 10089 8750 50  0000 C CNN
 F 2 "" H 10288 8600 50  0001 C CNN
@@
 AR Path="/5EAF7226/5F125E17" Ref="#PWR?"  Part="1"
 AR Path="/5EA98A67/5F125E17" Ref="#PWR?"  Part="1"
-AR Path="/5EA98353/5F125E17" Ref="#PWR019"  Part="1"
-F 0 "#PWR019" H 10250 8350 50  0001 C CNN
+AR Path="/5EA98353/5F125E17" Ref="#PWR?"  Part="1"
+F 0 "#PWR?" H 10250 8350 50  0001 C CNN
 F 1 "GND" H 10255 8427 50  0000 C CNN
 F 2 "" H 10250 8600 50  0001 C CNN
@@
 	10200 5400 10450 5400
 $Comp
-L power:GND #PWR?
-U 1 1 5F134BF9
-P 5150 3600
-AR Path="/5EAF7226/5F134BF9" Ref="#PWR?"  Part="1"
-AR Path="/5EA98A67/5F134BF9" Ref="#PWR?"  Part="1"
-AR Path="/5EA98353/5F134BF9" Ref="#PWR010"  Part="1"
-F 0 "#PWR010" H 5150 3350 50  0001 C CNN
-F 1 "GND" H 5155 3427 50  0000 C CNN
-F 2 "" H 5150 3600 50  0001 C CNN
-F 3 "" H 5150 3600 50  0001 C CNN
-	1    5150 3600
+L power:PWR_FLAG #FLG?
+U 1 1 5F13448F
+P 10450 5400
+AR Path="/5EA045EA/5F13448F" Ref="#FLG?"  Part="1"
+AR Path="/5EA98353/5EA34234/5F13448F" Ref="#FLG?"  Part="1"
+F 0 "#FLG?" H 10450 5475 50  0001 C CNN
+F 1 "PWR_FLAG" V 10450 5527 50  0000 L CNN
+F 2 "" H 10450 5400 50  0001 C CNN
+F 3 "~" H 10450 5400 50  0001 C CNN
+	1    10450 5400
 	0    1    1    0
 $EndComp
+$Comp
+L power:PWR_FLAG #FLG?
+U 1 1 5F13FFCB
+P 7150 3300
+AR Path="/5EA045EA/5F13FFCB" Ref="#FLG?"  Part="1"
+AR Path="/5EA98353/5EA34234/5F13FFCB" Ref="#FLG?"  Part="1"
+F 0 "#FLG?" H 7150 3375 50  0001 C CNN
+F 1 "PWR_FLAG" V 7150 3427 50  0000 L CNN
+F 2 "" H 7150 3300 50  0001 C CNN
+F 3 "~" H 7150 3300 50  0001 C CNN
+	1    7150 3300
+	0    -1   -1   0
+$EndComp
+$Comp
+L power:PWR_FLAG #FLG?
+U 1 1 5F14BDF0
+P 5400 5400
+AR Path="/5EA045EA/5F14BDF0" Ref="#FLG?"  Part="1"
+AR Path="/5EA98353/5EA34234/5F14BDF0" Ref="#FLG?"  Part="1"
+F 0 "#FLG?" H 5400 5475 50  0001 C CNN
+F 1 "PWR_FLAG" V 5400 5527 50  0000 L CNN
+F 2 "" H 5400 5400 50  0001 C CNN
+F 3 "~" H 5400 5400 50  0001 C CNN
+	1    5400 5400
+	0    1    1    0
+$EndComp
+$Comp
+L power:PWR_FLAG #FLG?
+U 1 1 5F156375
+P 5400 9000
+AR Path="/5EA045EA/5F156375" Ref="#FLG?"  Part="1"
+AR Path="/5EA98353/5EA34234/5F156375" Ref="#FLG?"  Part="1"
+F 0 "#FLG?" H 5400 9075 50  0001 C CNN
+F 1 "PWR_FLAG" V 5400 9127 50  0000 L CNN
+F 2 "" H 5400 9000 50  0001 C CNN
+F 3 "~" H 5400 9000 50  0001 C CNN
+	1    5400 9000
+	0    1    1    0
+$EndComp
+$Comp
+L power:PWR_FLAG #FLG?
+U 1 1 5F16E81F
+P 10450 9000
+AR Path="/5EA045EA/5F16E81F" Ref="#FLG?"  Part="1"
+AR Path="/5EA98353/5EA34234/5F16E81F" Ref="#FLG?"  Part="1"
+F 0 "#FLG?" H 10450 9075 50  0001 C CNN
+F 1 "PWR_FLAG" V 10450 9127 50  0000 L CNN
+F 2 "" H 10450 9000 50  0001 C CNN
+F 3 "~" H 10450 9000 50  0001 C CNN
+	1    10450 9000
+	0    1    1    0
+$EndComp
